Commit message: update jodell mesh path

File: urdf/fiveages_w1_leapmotor.urdf (robot description, URDF)
Before this commit: robot FiveAges W1, 44 links, 43 joints
Links:
- removed link left_left_driver
- removed link left_right_driver
- removed link right_left_driver
- removed link right_right_driver
- added link left_left_finger, mass 0.123532229208125; collision mesh filename=package://jodell_description/meshes/RG75/finger.obj; visual mesh filename=package://jodell_description/meshes/RG75/finger.obj
- added link left_right_finger, mass 0.123532779120439; collision mesh filename=package://jodell_description/meshes/RG75/finger.obj scale=-1 -1 1; visual mesh filename=package://jodell_description/meshes/RG75/finger.obj scale=-1 -1 1
- added link right_left_finger, mass 0.123532229208125; collision mesh filename=package://jodell_description/meshes/RG75/finger.obj; visual mesh filename=package://jodell_description/meshes/RG75/finger.obj
- added link right_right_finger, mass 0.123532779120439; collision mesh filename=package://jodell_description/meshes/RG75/finger.obj scale=-1 -1 1; visual mesh filename=package://jodell_description/meshes/RG75/finger.obj scale=-1 -1 1
- link left_flange: geometry collision mesh filename=package://jodell_description/meshes/RG75/flange.obj; visual mesh filename=package://jodell_description/meshes/RG75/flange.obj
- link left_gripper_base: geometry collision mesh filename=package://jodell_description/meshes/RG75/base.obj; visual mesh filename=package://jodell_description/meshes/RG75/base.obj
- link left_left_finger_pad: geometry collision mesh filename=package://jodell_description/meshes/RG75/pad_leapmotor.obj; visual mesh filename=package://jodell_description/meshes/RG75/pad_leapmotor.obj
- link left_right_finger_pad: geometry collision mesh filename=package://jodell_description/meshes/RG75/pad_leapmotor.obj scale=1 -1 1; visual mesh filename=package://jodell_description/meshes/RG75/pad_leapmotor.obj scale=1 -1 1
- link right_flange: geometry collision mesh filename=package://jodell_description/meshes/RG75/flange.obj; visual mesh filename=package://jodell_description/meshes/RG75/flange.obj
- link right_gripper_base: geometry collision mesh filename=package://jodell_description/meshes/RG75/base.obj; visual mesh filename=package://jodell_description/meshes/RG75/base.obj
- link right_left_finger_pad: geometry collision mesh filename=package://jodell_description/meshes/RG75/pad_leapmotor.obj; visual mesh filename=package://jodell_description/meshes/RG75/pad_leapmotor.obj
- link right_right_finger_pad: geometry collision mesh filename=package://jodell_description/meshes/RG75/pad_leapmotor.obj scale=1 -1 1; visual mesh filename=package://jodell_description/meshes/RG75/pad_leapmotor.obj scale=1 -1 1
- link trunk_base_link: geometry 
Joints:
- removed joint left_left_driver_joint
- removed joint right_left_driver_joint
- added joint left_right_finger_joint: type prismatic, parent left_gripper_base, child left_right_finger, origin xyz=-0.01475 -0.005263 0.13525, axis 0 -1 0, limit lower=-3.14 upper=3.14 effort=100 velocity=1, mimic joint=left_gripper_joint multiplier=1 offset=0
- added joint right_right_finger_joint: type prismatic, parent right_gripper_base, child right_right_finger, origin xyz=-0.01475 -0.005263 0.13525, axis 0 -1 0, limit lower=-3.14 upper=3.14 effort=100 velocity=1, mimic joint=right_gripper_joint multiplier=1 offset=0
- joint left_gripper_joint: axis 0 -1 0 -> 0 1 0; child left_right_driver -> left_left_finger; origin xyz=-0.01475 -0.005263 0.13525 -> xyz=0.01475 0.005263 0.13525
- joint left_left_finger_pad_joint: parent left_left_driver -> left_left_finger
- joint left_right_finger_pad_joint: parent left_right_driver -> left_right_finger
- joint right_gripper_joint: axis 0 -1 0 -> 0 1 0; child right_right_driver -> right_left_finger; origin xyz=-0.01475 -0.005263 0.13525 -> xyz=0.01475 0.005263 0.13525
- joint right_left_finger_pad_joint: parent right_left_driver -> right_left_finger
- joint right_right_finger_pad_joint: parent right_right_driver -> right_right_finger

File: urdf/fiveages_w1_rg75.urdf (robot description, URDF)
Before this commit: robot FiveAges W1, 44 links, 43 joints
Links:
- removed link left_left_driver
- removed link left_right_driver
- removed link right_left_driver
- removed link right_right_driver
- added link left_left_finger, mass 0.123532229208125; collision mesh filename=package://jodell_description/meshes/RG75/finger.obj; visual mesh filename=package://jodell_description/meshes/RG75/finger.obj
- added link left_right_finger, mass 0.123532779120439; collision mesh filename=package://jodell_description/meshes/RG75/finger.obj scale=-1 -1 1; visual mesh filename=package://jodell_description/meshes/RG75/finger.obj scale=-1 -1 1
- added link right_left_finger, mass 0.123532229208125; collision mesh filename=package://jodell_description/meshes/RG75/finger.obj; visual mesh filename=package://jodell_description/meshes/RG75/finger.obj
- added link right_right_finger, mass 0.123532779120439; collision mesh filename=package://jodell_description/meshes/RG75/finger.obj scale=-1 -1 1; visual mesh filename=package://jodell_description/meshes/RG75/finger.obj scale=-1 -1 1
- link base_link: geometry collision box size=.66 .55 .2; collision sphere radius=0.0365
- link body_link1: geometry collision mesh filename=package://fiveages_w1_description/meshes/body/link1.obj; visual mesh filename=package://fiveages_w1_description/meshes/body/link1.obj
- link body_link2: geometry collision mesh filename=package://fiveages_w1_description/meshes/body/link2.obj; visual mesh filename=package://fiveages_w1_description/meshes/body/link2.obj
- link body_link3: geometry collision mesh filename=package://fiveages_w1_description/meshes/body/link3.obj; visual mesh filename=package://fiveages_w1_description/meshes/body/link3.obj
- link body_link4: geometry collision mesh filename=package://fiveages_w1_description/meshes/body/link4.obj; visual mesh filename=package://fiveages_w1_description/meshes/body/link4.obj
- link chassis_left_Link: geometry collision cylinder length=0.038 radius=0.0842; visual mesh filename=package://fiveages_w1_description/meshes/chassis/wheel.obj
- link chassis_right_Link: geometry collision cylinder length=0.038 radius=0.0842; visual mesh filename=package://fiveages_w1_description/meshes/chassis/wheel.obj scale=1 -1 1
- link head_link1: geometry collision mesh filename=package://fiveages_w1_description/meshes/body/head1.obj; visual mesh filename=package://fiveages_w1_description/meshes/body/head1.obj
- link head_link2: geometry collision mesh filename=package://fiveages_w1_description/meshes/body/head2.obj; visual mesh filename=package://fiveages_w1_description/meshes/body/head2.obj
- link left_base_link: geometry collision mesh filename=package://rokae_ar5_description/meshes/base.obj scale=1 1 1; visual mesh filename=package://rokae_ar5_description/meshes/base.obj scale=1 1 1
- link left_flange: geometry collision mesh filename=package://jodell_description/meshes/RG75/flange.obj; visual mesh filename=package://jodell_description/meshes/RG75/flange.obj
- link left_gripper_base: geometry collision mesh filename=package://jodell_description/meshes/RG75/base.obj; visual mesh filename=package://jodell_description/meshes/RG75/base.obj
- link left_left_finger_pad: geometry collision mesh filename=package://jodell_description/meshes/RG75/pad_fiveages.obj; visual mesh filename=package://jodell_description/meshes/RG75/pad_fiveages.obj
- link left_link1: geometry collision mesh filename=package://rokae_ar5_description/meshes/link1.obj scale=1 1 1; visual mesh filename=package://rokae_ar5_description/meshes/link1.obj scale=1 1 1
- link left_link2: geometry collision mesh filename=package://rokae_ar5_description/meshes/link2.obj scale=1 1 1; visual mesh filename=package://rokae_ar5_description/meshes/link2.obj scale=1 1 1
- link left_link3: geometry collision mesh filename=package://rokae_ar5_description/meshes/link3.obj scale=1 1 1; visual mesh filename=package://rokae_ar5_description/meshes/link3.obj scale=1 1 1
- link left_link4: geometry collision mesh filename=package://rokae_ar5_description/meshes/link4.obj scale=1 1 1; visual mesh filename=package://rokae_ar5_description/meshes/link4.obj scale=1 1 1
- link left_link5: geometry collision mesh filename=package://rokae_ar5_description/meshes/link5.obj scale=1 1 1; visual mesh filename=package://rokae_ar5_description/meshes/link5.obj scale=1 1 1
- link left_link6: geometry collision mesh filename=package://rokae_ar5_description/meshes/link6.obj scale=1 1 1; visual mesh filename=package://rokae_ar5_description/meshes/link6.obj scale=1 1 1
- link left_link7: geometry collision mesh filename=package://rokae_ar5_description/meshes/link7.obj scale=1 1 1; visual mesh filename=package://rokae_ar5_description/meshes/link7.obj scale=1 1 1
- link left_right_finger_pad: geometry collision mesh filename=package://jodell_description/meshes/RG75/pad_fiveages.obj scale=1 -1 1; visual mesh filename=package://jodell_description/meshes/RG75/pad_fiveages.obj scale=1 -1 1
- link right_base_link: geometry collision mesh filename=package://rokae_ar5_description/meshes/base.obj scale=1 -1 1; visual mesh filename=package://rokae_ar5_description/meshes/base.obj scale=1 -1 1
- link right_flange: geometry collision mesh filename=package://jodell_description/meshes/RG75/flange.obj; visual mesh filename=package://jodell_description/meshes/RG75/flange.obj
- link right_gripper_base: geometry collision mesh filename=package://jodell_description/meshes/RG75/base.obj; visual mesh filename=package://jodell_description/meshes/RG75/base.obj
- link right_left_finger_pad: geometry collision mesh filename=package://jodell_description/meshes/RG75/pad_fiveages.obj; visual mesh filename=package://jodell_description/meshes/RG75/pad_fiveages.obj
- link right_link1: geometry collision mesh filename=package://rokae_ar5_description/meshes/link1.obj scale=1 -1 1; visual mesh filename=package://rokae_ar5_description/meshes/link1.obj scale=1 -1 1
- link right_link2: geometry collision mesh filename=package://rokae_ar5_description/meshes/link2.obj scale=1 -1 1; visual mesh filename=package://rokae_ar5_description/meshes/link2.obj scale=1 -1 1
- link right_link3: geometry collision mesh filename=package://rokae_ar5_description/meshes/link3.obj scale=1 -1 1; visual mesh filename=package://rokae_ar5_description/meshes/link3.obj scale=1 -1 1
- link right_link4: geometry collision mesh filename=package://rokae_ar5_description/meshes/link4.obj scale=1 -1 1; visual mesh filename=package://rokae_ar5_description/meshes/link4.obj scale=1 -1 1
- link right_link5: geometry collision mesh filename=package://rokae_ar5_description/meshes/link5.obj scale=1 -1 1; visual mesh filename=package://rokae_ar5_description/meshes/link5.obj scale=1 -1 1
- link right_link6: geometry collision mesh filename=package://rokae_ar5_description/meshes/link6.obj scale=1 -1 1; visual mesh filename=package://rokae_ar5_description/meshes/link6.obj scale=1 -1 1
- link right_link7: geometry collision mesh filename=package://rokae_ar5_description/meshes/link7.obj scale=1 -1 1; visual mesh filename=package://rokae_ar5_description/meshes/link7.obj scale=1 -1 1
- link right_right_finger_pad: geometry collision mesh filename=package://jodell_description/meshes/RG75/pad_fiveages.obj scale=1 -1 1; visual mesh filename=package://jodell_description/meshes/RG75/pad_fiveages.obj scale=1 -1 1
- link trunk_base_link: geometry 
Joints:
- removed joint left_left_driver_joint
- removed joint right_left_driver_joint
- added joint left_right_finger_joint: type prismatic, parent left_gripper_base, child left_right_finger, origin xyz=-0.01475 -0.005263 0.13525, axis 0 -1 0, limit lower=-3.14 upper=3.14 effort=100 velocity=1, mimic joint=left_gripper_joint multiplier=1 offset=0
- added joint right_right_finger_joint: type prismatic, parent right_gripper_base, child right_right_finger, origin xyz=-0.01475 -0.005263 0.13525, axis 0 -1 0, limit lower=-3.14 upper=3.14 effort=100 velocity=1, mimic joint=right_gripper_joint multiplier=1 offset=0
- joint left_gripper_joint: axis 0 -1 0 -> 0 1 0; child left_right_driver -> left_left_finger; origin xyz=-0.01475 -0.005263 0.13525 -> xyz=0.01475 0.005263 0.13525
- joint left_left_finger_pad_joint: parent left_left_driver -> left_left_finger
- joint left_right_finger_pad_joint: parent left_right_driver -> left_right_finger
- joint right_gripper_joint: axis 0 -1 0 -> 0 1 0; child right_right_driver -> right_left_finger; origin xyz=-0.01475 -0.005263 0.13525 -> xyz=0.01475 0.005263 0.13525
- joint right_left_finger_pad_joint: parent right_left_driver -> right_left_finger
- joint right_right_finger_pad_joint: parent right_right_driver -> right_right_finger
