Commit message: 增加Linkhou & leapmotor的组合 urdf文件中的filename改成package形式

File: urdf/fiveages_w1_linkhou_rg75.urdf (robot description, URDF)
Before this commit: robot FiveAges W1, 43 links, 42 joints
Links:
- link base_link: geometry collision box size=0.5796094 0.449 0.27073438; collision sphere radius=0.038
- link body_link1: geometry collision mesh filename=package://fiveages_w1_description/meshes/body/link1.obj; visual mesh filename=package://fiveages_w1_description/meshes/body/link1.obj
- link body_link2: geometry collision mesh filename=package://fiveages_w1_description/meshes/body/link2.obj; visual mesh filename=package://fiveages_w1_description/meshes/body/link2.obj
- link body_link3: geometry collision mesh filename=package://fiveages_w1_description/meshes/body/link3.obj; visual mesh filename=package://fiveages_w1_description/meshes/body/link3.obj
- link body_link4: geometry collision mesh filename=package://fiveages_w1_description/meshes/body/link4.obj; visual mesh filename=package://fiveages_w1_description/meshes/body/link4.obj
- link head_link1: geometry collision mesh filename=package://fiveages_w1_description/meshes/body/head1.obj; visual mesh filename=package://fiveages_w1_description/meshes/body/head1.obj
- link head_link2: geometry collision mesh filename=package://fiveages_w1_description/meshes/body/head2.obj; visual mesh filename=package://fiveages_w1_description/meshes/body/head2.obj
- link left_base_link: geometry collision mesh filename=package://rokae_ar5_description/meshes/base.obj scale=1 1 1; visual mesh filename=package://rokae_ar5_description/meshes/base.obj scale=1 1 1
- link left_flange: geometry collision mesh filename=package://jodell_description/meshes/RG75/flange.obj; visual mesh filename=package://jodell_description/meshes/RG75/flange.obj
- link left_gripper_base: geometry collision mesh filename=package://jodell_description/meshes/RG75/base.obj; visual mesh filename=package://jodell_description/meshes/RG75/base.obj
- link left_left_finger: geometry collision mesh filename=package://jodell_description/meshes/RG75/finger.obj; visual mesh filename=package://jodell_description/meshes/RG75/finger.obj
- link left_left_finger_pad: geometry collision mesh filename=package://jodell_description/meshes/RG75/pad_fiveages.obj; visual mesh filename=package://jodell_description/meshes/RG75/pad_fiveages.obj
- link left_link1: geometry collision mesh filename=package://rokae_ar5_description/meshes/link1.obj scale=1 1 1; visual mesh filename=package://rokae_ar5_description/meshes/link1.obj scale=1 1 1
- link left_link2: geometry collision mesh filename=package://rokae_ar5_description/meshes/link2.obj scale=1 1 1; visual mesh filename=package://rokae_ar5_description/meshes/link2.obj scale=1 1 1
- link left_link3: geometry collision mesh filename=package://rokae_ar5_description/meshes/link3.obj scale=1 1 1; visual mesh filename=package://rokae_ar5_description/meshes/link3.obj scale=1 1 1
- link left_link4: geometry collision mesh filename=package://rokae_ar5_description/meshes/link4.obj scale=1 1 1; visual mesh filename=package://rokae_ar5_description/meshes/link4.obj scale=1 1 1
- link left_link5: geometry collision mesh filename=package://rokae_ar5_description/meshes/link5.obj scale=1 1 1; visual mesh filename=package://rokae_ar5_description/meshes/link5.obj scale=1 1 1
- link left_link6: geometry collision mesh filename=package://rokae_ar5_description/meshes/link6.obj scale=1 1 1; visual mesh filename=package://rokae_ar5_description/meshes/link6.obj scale=1 1 1
- link left_link7: geometry collision mesh filename=package://rokae_ar5_description/meshes/link7.obj scale=1 1 1; visual mesh filename=package://rokae_ar5_description/meshes/link7.obj scale=1 1 1
- link left_right_finger: geometry collision mesh filename=package://jodell_description/meshes/RG75/finger.obj scale=-1 -1 1; visual mesh filename=package://jodell_description/meshes/RG75/finger.obj scale=-1 -1 1
- link left_right_finger_pad: geometry collision mesh filename=package://jodell_description/meshes/RG75/pad_fiveages.obj scale=1 -1 1; visual mesh filename=package://jodell_description/meshes/RG75/pad_fiveages.obj scale=1 -1 1
- link left_wheel: geometry collision cylinder length=0.036 radius=0.07948; visual mesh filename=package://fiveages_w1_description/meshes/linkhou_q1/wheel.o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
- link right_base_link: geometry collision mesh filename=package://rokae_ar5_description/meshes/base.obj scale=1 -1 1; visual mesh filename=package://rokae_ar5_description/meshes/base.obj scale=1 -1 1
- link right_flange: geometry collision mesh filename=package://jodell_description/meshes/RG75/flange.obj; visual mesh filename=package://jodell_description/meshes/RG75/flange.obj
- link right_gripper_base: geometry collision mesh filename=package://jodell_description/meshes/RG75/base.obj; visual mesh filename=package://jodell_description/meshes/RG75/base.obj
- link right_left_finger: geometry collision mesh filename=package://jodell_description/meshes/RG75/finger.obj; visual mesh filename=package://jodell_description/meshes/RG75/finger.obj
- link right_left_finger_pad: geometry collision mesh filename=package://jodell_description/meshes/RG75/pad_fiveages.obj; visual mesh filename=package://jodell_description/meshes/RG75/pad_fiveages.obj
- link right_link1: geometry collision mesh filename=package://rokae_ar5_description/meshes/link1.obj scale=1 -1 1; visual mesh filename=package://rokae_ar5_description/meshes/link1.obj scale=1 -1 1
- link right_link2: geometry collision mesh filename=package://rokae_ar5_description/meshes/link2.obj scale=1 -1 1; visual mesh filename=package://rokae_ar5_description/meshes/link2.obj scale=1 -1 1
- link right_link3: geometry collision mesh filename=package://rokae_ar5_description/meshes/link3.obj scale=1 -1 1; visual mesh filename=package://rokae_ar5_description/meshes/link3.obj scale=1 -1 1
- link right_link4: geometry collision mesh filename=package://rokae_ar5_description/meshes/link4.obj scale=1 -1 1; visual mesh filename=package://rokae_ar5_description/meshes/link4.obj scale=1 -1 1
- link right_link5: geometry collision mesh filename=package://rokae_ar5_description/meshes/link5.obj scale=1 -1 1; visual mesh filename=package://rokae_ar5_description/meshes/link5.obj scale=1 -1 1
- link right_link6: geometry collision mesh filename=package://rokae_ar5_description/meshes/link6.obj scale=1 -1 1; visual mesh filename=package://rokae_ar5_description/meshes/link6.obj scale=1 -1 1
- link right_link7: geometry collision mesh filename=package://rokae_ar5_description/meshes/link7.obj scale=1 -1 1; visual mesh filename=package://rokae_ar5_description/meshes/link7.obj scale=1 -1 1
- link right_right_finger: geometry collision mesh filename=package://jodell_description/meshes/RG75/finger.obj scale=-1 -1 1; visual mesh filename=package://jodell_description/meshes/RG75/finger.obj scale=-1 -1 1
- link right_right_finger_pad: geometry collision mesh filename=package://jodell_description/meshes/RG75/pad_fiveages.obj scale=1 -1 1; visual mesh filename=package://jodell_description/meshes/RG75/pad_fiveages.obj scale=1 -1 1
- link right_wheel: geometry collision cylinder length=0.036 radius=0.07948; visual mesh filename=package://fiveages_w1_description/meshes/linkhou_q1/wheel.o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 scale=1 -1 1

File: xacro/robot.xacro (robot description, xacro)
@@ -10,4 +10,8 @@
 		<xacro:property name="selected_chassis" value="linkhou_q1"/>
 		<xacro:property name="selected_gripper_type" value="rg75"/>
+	</xacro:if>
+	<xacro:if value="${type_arg == 'linkhou_leapmotor'}">
+		<xacro:property name="selected_chassis" value="linkhou_q1"/>
+		<xacro:property name="selected_gripper_type" value="leapmotor"/>
 	</xacro:if>
 	<!-- Include Component Macros -->

File: xacro/ros2_control/robot.xacro (robot description, xacro)
@@ -7,4 +7,17 @@
     <xacro:include filename="$(find fiveages_w1_description)/xacro/ros2_control/body.xacro"/>
     <xacro:include filename="$(find fiveages_w1_description)/xacro/ros2_control/chassis.xacro"/>
+    <xacro:property name="ros2_control_config_basename" value="ros2_controllers.yaml"/>
+    <xacro:if value="${type_arg == 'rg75'}">
+        <xacro:property name="ros2_control_config_basename" value="rg75.yaml"/>
+    </xacro:if>
+    <xacro:if value="${type_arg == 'leapmotor'}">
+        <xacro:property name="ros2_control_config_basename" value="leapmotor.yaml"/>
+    </xacro:if>
+    <xacro:if value="${type_arg == 'linkhou_rg75'}">
+        <xacro:property name="ros2_control_config_basename" value="linkhou_rg75.yaml"/>
+    </xacro:if>
+    <xacro:if value="${type_arg == 'linkhou_leapmotor'}">
+        <xacro:property name="ros2_control_config_basename" value="linkhou_leapmotor.yaml"/>
+    </xacro:if>
     <xacro:if value="${'$(arg ros2_control_hardware_type)' == 'real'}">
         <ros2_control name="ar5_left_system" type="system">
@@ -65,5 +78,5 @@
             <xacro:ar5_interfaces name="left"/>
             <xacro:ar5_interfaces name="right"/>
-            <xacro:if value="${'$(arg type)' == 'rg75' or '$(arg type)' == 'leapmotor' or '$(arg type)' == 'linkhou_rg75'}">
+            <xacro:if value="${'$(arg type)' == 'rg75' or '$(arg type)' == 'leapmotor' or '$(arg type)' == 'linkhou_rg75' or '$(arg type)' == 'linkhou_leapmotor'}">
                 <xacro:include filename="$(find jodell_description)/xacro/ros2_control/RG75-300.xacro"/>
                 <xacro:rg75_interfaces name="left"/>
@@ -77,5 +90,5 @@
         <gazebo>
             <plugin filename="gz_ros2_control-system" name="gz_ros2_control::GazeboSimROS2ControlPlugin">
-                <parameters>$(find fiveages_w1_description)/config/ros2_control/ros2_controllers.yaml</parameters>
+                <parameters>$(find fiveages_w1_description)/config/ros2_control/${ros2_control_config_basename}</parameters>
             </plugin>
         </gazebo>
