Commit message: 修复ocs2中marker初始状态和eef不对齐

File: urdf/fiveages_w1_rg75.urdf (robot description, URDF)
Before this commit: robot FiveAges W1, 44 links, 43 joints
Joints:
- joint body_joint1: axis 0 -1 0 -> 0 1 0; limit lower=-2.57 upper=2.57 effort=300 velocity=15 -> lower=0 upper=1.504 effort=300 velocity=15
- joint body_joint2: axis 0 -1 0 -> 0 1 0; limit lower=-3.14 upper=3.14 effort=300 velocity=15 -> lower=-2.5 upper=2.5 effort=300 velocity=15
- joint body_joint3: axis 0 1 0 -> 0 -1 0; limit lower=-3.14 upper=3.14 effort=300 velocity=15 -> lower=-3.14 upper=0 effort=300 velocity=15
- joint left_gripper_base_joint: origin (none) -> xyz=0 0 -0.0045
- joint left_joint1: limit lower=-3.1414 upper=3.1414 effort=108 velocity=3.9269908169872414 -> lower=-3.14 upper=3.14 effort=108 velocity=3.9269908169872414
- joint left_joint2: limit lower=-2.1293 upper=2.1293 effort=108 velocity=3.9269908169872414 -> lower=-2.12 upper=2.12 effort=108 velocity=3.9269908169872414
- joint left_joint3: limit lower=-3.1416 upper=3.1416 effort=66 velocity=5.235987755982989 -> lower=-3.14 upper=3.14 effort=66 velocity=5.235987755982989
- joint left_joint4: limit lower=-1.3963 upper=2.5307 effort=66 velocity=5.235987755982989 -> lower=-1.39 upper=2.50 effort=66 velocity=5.235987755982989
- joint left_joint5: limit lower=-3.1416 upper=3.1416 effort=19 velocity=4.1887902047863905 -> lower=-3.14 upper=3.14 effort=19 velocity=4.1887902047863905
- joint left_joint6: limit lower=-1.9722 upper=1.9722 effort=19 velocity=4.1887902047863905 -> lower=-1.96 upper=1.96 effort=19 velocity=4.1887902047863905
- joint left_joint7: limit lower=-3.1416 upper=3.1416 effort=19 velocity=4.1887902047863905 -> lower=-3.14 upper=3.14 effort=19 velocity=4.1887902047863905
- joint right_joint1: limit lower=-3.1414 upper=3.1414 effort=108 velocity=3.9269908169872414 -> lower=-3.14 upper=3.14 effort=108 velocity=3.9269908169872414
- joint right_joint2: limit lower=-2.1293 upper=2.1293 effort=108 velocity=3.9269908169872414 -> lower=-2.12 upper=2.12 effort=108 velocity=3.9269908169872414
- joint right_joint3: limit lower=-3.1416 upper=3.1416 effort=66 velocity=5.235987755982989 -> lower=-3.14 upper=3.14 effort=66 velocity=5.235987755982989
- joint right_joint4: limit lower=-1.3963 upper=2.5307 effort=66 velocity=5.235987755982989 -> lower=-1.39 upper=2.50 effort=66 velocity=5.235987755982989
- joint right_joint5: limit lower=-3.1416 upper=3.1416 effort=19 velocity=4.1887902047863905 -> lower=-3.14 upper=3.14 effort=19 velocity=4.1887902047863905
- joint right_joint6: limit lower=-1.9722 upper=1.9722 effort=19 velocity=4.1887902047863905 -> lower=-1.96 upper=1.96 effort=19 velocity=4.1887902047863905
- joint right_joint7: limit lower=-3.1416 upper=3.1416 effort=19 velocity=4.1887902047863905 -> lower=-3.14 upper=3.14 effort=19 velocity=4.1887902047863905
