Commit message: add linkhou q1

File: urdf/fiveages_w1.urdf (robot description, URDF)
Before this commit: robot FiveAges W1, 30 links, 29 joints
Joints:
- joint body_joint1: limit lower=-1.57 upper=1.57 effort=300 velocity=15 -> lower=-2.57 upper=2.57 effort=300 velocity=15
- joint body_joint2: limit lower=-1.57 upper=1.57 effort=300 velocity=15 -> lower=-3.14 upper=3.14 effort=300 velocity=15
- joint body_joint3: limit lower=-1.57 upper=1.57 effort=300 velocity=15 -> lower=-3.14 upper=3.14 effort=300 velocity=15
- joint body_joint4: limit lower=-1.57 upper=1.57 effort=300 velocity=15 -> lower=-3.14 upper=3.14 effort=300 velocity=15

File: urdf/fiveages_w1_leapmotor.urdf (robot description, URDF)
Before this commit: robot FiveAges W1, 44 links, 43 joints
Joints:
- joint body_joint1: limit lower=-1.57 upper=1.57 effort=300 velocity=15 -> lower=-2.57 upper=2.57 effort=300 velocity=15
- joint body_joint2: limit lower=-1.57 upper=1.57 effort=300 velocity=15 -> lower=-3.14 upper=3.14 effort=300 velocity=15
- joint body_joint3: limit lower=-1.57 upper=1.57 effort=300 velocity=15 -> lower=-3.14 upper=3.14 effort=300 velocity=15
- joint body_joint4: limit lower=-1.57 upper=1.57 effort=300 velocity=15 -> lower=-3.14 upper=3.14 effort=300 velocity=15

File: urdf/fiveages_w1_rg75.urdf (robot description, URDF)
Before this commit: robot FiveAges W1, 44 links, 43 joints
Joints:
- joint body_joint1: limit lower=-1.57 upper=1.57 effort=300 velocity=15 -> lower=-2.57 upper=2.57 effort=300 velocity=15
- joint body_joint2: limit lower=-1.57 upper=1.57 effort=300 velocity=15 -> lower=-3.14 upper=3.14 effort=300 velocity=15
- joint body_joint3: limit lower=-1.57 upper=1.57 effort=300 velocity=15 -> lower=-3.14 upper=3.14 effort=300 velocity=15
- joint body_joint4: limit lower=-1.57 upper=1.57 effort=300 velocity=15 -> lower=-3.14 upper=3.14 effort=300 velocity=15

File: xacro/body.xacro (robot description, xacro)
@@ -52,5 +52,5 @@
             <child link="body_link1"/>
             <axis xyz="0 -1 0"/>
-            <limit lower="-1.57" upper="1.57" effort="300" velocity="15"/>
+            <limit lower="-3.14" upper="3.14" effort="300" velocity="15"/>
             <dynamics damping="0.01" friction="0.1"/>
         </joint>
@@ -83,5 +83,5 @@
             <child link="body_link2"/>
             <axis xyz="0 -1 0"/>
-            <limit lower="-1.57" upper="1.57" effort="300" velocity="15"/>
+            <limit lower="-3.14" upper="3.14" effort="300" velocity="15"/>
             <dynamics damping="0.01" friction="0.1"/>
         </joint>
@@ -114,5 +114,5 @@
             <child link="body_link3"/>
             <axis xyz="0 1 0"/>
-            <limit lower="-1.57" upper="1.57" effort="300" velocity="15"/>
+            <limit lower="-3.14" upper="3.14" effort="300" velocity="15"/>
             <dynamics damping="0.01" friction="0.1"/>
         </joint>
@@ -145,5 +145,5 @@
             <child link="body_link4"/>
             <axis xyz="0 0 1"/>
-            <limit lower="-1.57" upper="1.57" effort="300" velocity="15"/>
+            <limit lower="-3.14" upper="3.14" effort="300" velocity="15"/>
             <dynamics damping="0.01" friction="0.1"/>
         </joint>

File: xacro/robot.xacro (robot description, xacro)
@@ -2,5 +2,5 @@
 <robot name="FiveAges W1" xmlns:xacro="http://www.ros.org/wiki/xacro">
 	<!-- Include Component Macros -->
-	<xacro:include filename="$(find fiveages_w1_description)/xacro/chassis.xacro"/>
+	<xacro:include filename="$(find fiveages_w1_description)/xacro/chassis/chassis.xacro"/>
 	<xacro:include filename="$(find fiveages_w1_description)/xacro/body.xacro"/>
 	<xacro:include filename="$(find rokae_ar5_description)/xacro/arm.xacro"/>

Commit message: deploy config for real robot with body joint

File: urdf/fiveages_w1.urdf (robot description, URDF)
Before this commit: robot FiveAges W1, 30 links, 29 joints
Links:
- added link left_eef
- added link right_eef
- link trunk_base_link: geometry 
Joints:
- added joint left_eef_joint: type fixed, parent left_link7, child left_eef
- added joint right_eef_joint: type fixed, parent right_link7, child right_eef
- joint body_joint1: axis 0 -1 0 -> 0 1 0; limit lower=-2.57 upper=2.57 effort=300 velocity=15 -> lower=-3.14 upper=3.14 effort=300 velocity=15
- joint body_joint2: axis 0 -1 0 -> 0 1 0
- joint body_joint3: axis 0 1 0 -> 0 -1 0

File: xacro/body.xacro (robot description, xacro)
@@ -51,5 +51,5 @@
             <parent link="trunk_base_link"/>
             <child link="body_link1"/>
-            <axis xyz="0 -1 0"/>
+            <axis xyz="0 1 0"/>
             <limit lower="-3.14" upper="3.14" effort="300" velocity="15"/>
             <dynamics damping="0.01" friction="0.1"/>
@@ -82,5 +82,5 @@
             <parent link="body_link1"/>
             <child link="body_link2"/>
-            <axis xyz="0 -1 0"/>
+            <axis xyz="0 1 0"/>
             <limit lower="-3.14" upper="3.14" effort="300" velocity="15"/>
             <dynamics damping="0.01" friction="0.1"/>
@@ -113,5 +113,5 @@
             <parent link="body_link2"/>
             <child link="body_link3"/>
-            <axis xyz="0 1 0"/>
+            <axis xyz="0 -1 0"/>
             <limit lower="-3.14" upper="3.14" effort="300" velocity="15"/>
             <dynamics damping="0.01" friction="0.1"/>

File: xacro/ros2_control/robot.xacro (robot description, xacro)
@@ -22,4 +22,19 @@
             <xacro:ar5_interfaces name="right"/>
         </ros2_control>
+        <ros2_control name="eyou_body" type="system">
+            <hardware>
+                <plugin>eyou_ros2_control/EyouHardware</plugin>
+                <param name="device_type">Canable</param>
+                <param name="device_index">0</param>
+                <param name="baudrate">1000</param>
+                <param name="motor_ids">[1, 2, 3, 4, 5, 6]</param>
+                <param name="control_period_ms">4</param>
+                <param name="report_period_ms">100</param>
+                <param name="use_sync">true</param>
+                <!-- 每个电机的减速比配置 -->
+                <param name="reduction_ratios">[121.0, 121.0, 121.0, 121.0, 56.0, 36.0]</param>
+            </hardware>
+            <xacro:body_interfaces/>
+        </ros2_control>
         <ros2_control name="virtual_system" type="system">
             <hardware>
@@ -27,5 +42,4 @@
             </hardware>
             <xacro:chassis_interfaces/>
-            <xacro:body_interfaces/>
         </ros2_control>
     </xacro:if>

Commit message: config for impedence control

File: urdf/fiveages_w1.urdf (robot description, URDF)
Before this commit: robot FiveAges W1, 32 links, 31 joints
Joints:
- joint body_joint1: limit lower=-3.14 upper=3.14 effort=300 velocity=15 -> lower=0.0 upper=1.504 effort=300 velocity=15
- joint body_joint2: limit lower=-3.14 upper=3.14 effort=300 velocity=15 -> lower=-2.5 upper=2.5 effort=300 velocity=15
- joint body_joint3: limit lower=-3.14 upper=3.14 effort=300 velocity=15 -> lower=-3.14 upper=0 effort=300 velocity=15

File: xacro/body.xacro (robot description, xacro)
@@ -52,5 +52,5 @@
             <child link="body_link1"/>
             <axis xyz="0 1 0"/>
-            <limit lower="-3.14" upper="3.14" effort="300" velocity="15"/>
+            <limit lower="0" upper="1.504" effort="300" velocity="15"/>
             <dynamics damping="0.01" friction="0.1"/>
         </joint>
@@ -83,5 +83,5 @@
             <child link="body_link2"/>
             <axis xyz="0 1 0"/>
-            <limit lower="-3.14" upper="3.14" effort="300" velocity="15"/>
+            <limit lower="-2.5" upper="2.5" effort="300" velocity="15"/>
             <dynamics damping="0.01" friction="0.1"/>
         </joint>
@@ -114,5 +114,5 @@
             <child link="body_link3"/>
             <axis xyz="0 -1 0"/>
-            <limit lower="-3.14" upper="3.14" effort="300" velocity="15"/>
+            <limit lower="-3.14" upper="0" effort="300" velocity="15"/>
             <dynamics damping="0.01" friction="0.1"/>
         </joint>

File: xacro/ros2_control/robot.xacro (robot description, xacro)
@@ -12,4 +12,5 @@
                 <plugin>rokae_ros2_control/RokaeHardware</plugin>
                 <param name="arm_ip">192.168.2.160</param>
+                <param name="joint_impedance">500,500,500,500,50,50,50</param>
             </hardware>
             <xacro:ar5_interfaces name="left"/>
@@ -19,4 +20,5 @@
                 <plugin>rokae_ros2_control/RokaeHardware</plugin>
                 <param name="arm_ip">192.168.2.161</param>
+                <param name="joint_impedance">500,500,500,500,50,50,50</param>
             </hardware>
             <xacro:ar5_interfaces name="right"/>
