Commit message: urdf fix

File: urdf/fiveages_w1.urdf (robot description, URDF)
Before this commit: robot FiveAges W1, 32 links, 31 joints
Links:
- link left_base_link: geometry collision mesh filename=package://rokae_ar5_description/meshes/srs/base.obj scale=1 1 1; visual mesh filename=package://rokae_ar5_description/meshes/srs/base.obj scale=1 1 1
- link left_link1: geometry collision mesh filename=package://rokae_ar5_description/meshes/srs/link1.obj scale=1 1 1; visual mesh filename=package://rokae_ar5_description/meshes/srs/link1.obj scale=1 1 1
- link left_link2: geometry collision mesh filename=package://rokae_ar5_description/meshes/srs/link2.obj scale=1 1 1; visual mesh filename=package://rokae_ar5_description/meshes/srs/link2.obj scale=1 1 1
- link left_link3: geometry collision mesh filename=package://rokae_ar5_description/meshes/srs/link3.obj scale=1 1 1; visual mesh filename=package://rokae_ar5_description/meshes/srs/link3.obj scale=1 1 1
- link left_link4: geometry collision mesh filename=package://rokae_ar5_description/meshes/srs/link4.obj scale=1 1 1; visual mesh filename=package://rokae_ar5_description/meshes/srs/link4.obj scale=1 1 1
- link left_link5: geometry collision mesh filename=package://rokae_ar5_description/meshes/srs/link5.obj scale=1 1 1; visual mesh filename=package://rokae_ar5_description/meshes/srs/link5.obj scale=1 1 1
- link left_link6: geometry collision mesh filename=package://rokae_ar5_description/meshes/srs/link6.obj scale=1 1 1; visual mesh filename=package://rokae_ar5_description/meshes/srs/link6.obj scale=1 1 1
- link left_link7: geometry collision mesh filename=package://rokae_ar5_description/meshes/srs/link7.obj scale=1 1 1; visual mesh filename=package://rokae_ar5_description/meshes/srs/link7.obj scale=1 1 1
- link right_base_link: geometry collision mesh filename=package://rokae_ar5_description/meshes/srs/base.obj scale=1 -1 1; visual mesh filename=package://rokae_ar5_description/meshes/srs/base.obj scale=1 -1 1
- link right_link1: geometry collision mesh filename=package://rokae_ar5_description/meshes/srs/link1.obj scale=1 -1 1; visual mesh filename=package://rokae_ar5_description/meshes/srs/link1.obj scale=1 -1 1
- link right_link2: geometry collision mesh filename=package://rokae_ar5_description/meshes/srs/link2.obj scale=1 -1 1; visual mesh filename=package://rokae_ar5_description/meshes/srs/link2.obj scale=1 -1 1
- link right_link3: geometry collision mesh filename=package://rokae_ar5_description/meshes/srs/link3.obj scale=1 -1 1; visual mesh filename=package://rokae_ar5_description/meshes/srs/link3.obj scale=1 -1 1
- link right_link4: geometry collision mesh filename=package://rokae_ar5_description/meshes/srs/link4.obj scale=1 -1 1; visual mesh filename=package://rokae_ar5_description/meshes/srs/link4.obj scale=1 -1 1
- link right_link5: geometry collision mesh filename=package://rokae_ar5_description/meshes/srs/link5.obj scale=1 -1 1; visual mesh filename=package://rokae_ar5_description/meshes/srs/link5.obj scale=1 -1 1
- link right_link6: geometry collision mesh filename=package://rokae_ar5_description/meshes/srs/link6.obj scale=1 -1 1; visual mesh filename=package://rokae_ar5_description/meshes/srs/link6.obj scale=1 -1 1
- link right_link7: geometry collision mesh filename=package://rokae_ar5_description/meshes/srs/link7.obj scale=1 -1 1; visual mesh filename=package://rokae_ar5_description/meshes/srs/link7.obj scale=1 -1 1

File: xacro/chassis/linkhou_q1.xacro (robot description, xacro)
@@ -86,10 +86,9 @@
             </collision>
         </link>
-        <joint name="chassis_left_joint" type="revolute">
+        <joint name="chassis_left_joint" type="continuous">
             <origin xyz="-0.026651 0.20625 ${drive_wheel_height}"/>
             <parent link="base_link"/>
             <child link="left_wheel"/>
             <axis xyz="0 1 0"/>
-            <limit lower="-3.14" upper="3.14" effort="100" velocity="1"/>
         </joint>
         <link name="right_wheel">
@@ -117,10 +116,9 @@
             </collision>
         </link>
-        <joint name="chassis_right_joint" type="revolute">
+        <joint name="chassis_right_joint" type="continuous">
             <origin xyz="-0.026651 -0.20625 ${drive_wheel_height}"/>
             <parent link="base_link"/>
             <child link="right_wheel"/>
-            <axis xyz="0 -1 0"/>
-            <limit lower="-3.14" upper="3.14" effort="100" velocity="1"/>
+            <axis xyz="0 1 0"/>
         </joint>
         <link name="scan"/>

File: xacro/component.xacro (robot description, xacro)
@@ -4,5 +4,5 @@
 <!-- |    This file includes the base robot structure and both arms                    | -->
 <!-- =================================================================================== -->
-<robot name="Fiveages_W1" xmlns:xacro="http://www.ros.org/wiki/xacro">
+<robot name="FiveAges_W1" xmlns:xacro="http://www.ros.org/wiki/xacro">
 	<xacro:arg name="type" default="base"/>
 	<xacro:if value="${'$(arg type)' == 'base'}">

File: xacro/robot.xacro (robot description, xacro)
@@ -19,5 +19,5 @@
 	<xacro:include filename="$(find fiveages_w1_description)/xacro/chassis/${selected_chassis}.xacro"/>
 	<xacro:include filename="$(find fiveages_w1_description)/xacro/body.xacro"/>
-	<xacro:include filename="$(find rokae_ar5_description)/xacro/arm.xacro"/>
+	<xacro:include filename="$(find rokae_ar5_description)/xacro/arm_srs.xacro"/>
 	<xacro:include filename="$(find fiveages_w1_description)/xacro/grippers.xacro"/>
 	<!-- Chassis -->

File: xacro/ros2_control/robot.xacro (robot description, xacro)
@@ -1,176 +1,179 @@
 <?xml version="1.0"?>
 <robot name="fiveages_w1" xmlns:xacro="http://www.ros.org/wiki/xacro">
-    <xacro:arg name="ros2_control_hardware_type" default="mock_components"/>
-    <!-- 直接include robot.xacro并根据type参数传递 -->
-    <xacro:include filename="$(find fiveages_w1_description)/xacro/robot.xacro"/>
-    <xacro:include filename="$(find rokae_ar5_description)/xacro/ros2_control/interfaces.xacro"/>
-    <xacro:include filename="$(find fiveages_w1_description)/xacro/ros2_control/body.xacro"/>
-    <xacro:include filename="$(find fiveages_w1_description)/xacro/ros2_control/chassis.xacro"/>
-    <xacro:if value="${'$(arg ros2_control_hardware_type)' == 'real'}">
-        <ros2_control name="ar5_left_system" type="system">
-            <hardware>
-                <plugin>rokae_ros2_control/RokaeHardware</plugin>
-                <param name="arm_ip">192.168.2.160</param>
-                <param name="joint_impedance">500,500,500,500,50,50,50</param>
-                <param name="local_ip">192.168.2.100</param>
-            </hardware>
-            <xacro:ar5_interfaces name="left"/>
-            <xacro:if value="${'$(arg type)' == 'rg75'}">
-                <joint name="left_gripper_joint">
-                    <command_interface name="position"/>
-                    <state_interface name="position">
-                        <param name="initial_value">0</param>
-                    </state_interface>
-                </joint>
-            </xacro:if>
-        </ros2_control>
-        <ros2_control name="ar5_right_system" type="system">
-            <hardware>
-                <plugin>rokae_ros2_control/RokaeHardware</plugin>
-                <param name="arm_ip">192.168.2.161</param>
-                <param name="joint_impedance">500,500,500,500,50,50,50</param>
-                <param name="local_ip">192.168.2.100</param>
-            </hardware>
-            <xacro:ar5_interfaces name="right"/>
-            <xacro:if value="${'$(arg type)' == 'rg75'}">
-                <joint name="right_gripper_joint">
-                    <command_interface name="position"/>
-                    <state_interface name="position">
-                        <param name="initial_value">0</param>
-                    </state_interface>
-                </joint>
-            </xacro:if>
-        </ros2_control>
-        <ros2_control name="eyou_body" type="system">
-            <hardware>
-                <plugin>eyou_ros2_control/EyouHardware</plugin>
-                <param name="device_type">Canable</param>
-                <param name="device_index">2 </param>
-                <param name="baudrate">1000</param>
-                <param name="motor_ids">[1, 2, 3, 4, 5, 6]</param>
-                <param name="control_period_ms">4</param>
-                <param name="report_period_ms">100</param>
-                <param name="use_sync">true</param>
-                <!-- 每个电机的减速比配置 -->
-                <param name="reduction_ratios">[121.0, 121.0, 121.0, 121.0, 56.0, 36.0]</param>
-            </hardware>
-            <xacro:body_interfaces/>
-        </ros2_control>
-        <ros2_control name="virtual_system" type="system">
-            <hardware>
-                <plugin>mock_components/GenericSystem</plugin>
-            </hardware>
-            <xacro:chassis_interfaces/>
-        </ros2_control>
-    </xacro:if>
-    <xacro:if value="${'$(arg ros2_control_hardware_type)' == 'real-laptop'}">
-        <ros2_control name="ar5_left_system" type="system">
-            <hardware>
-                <plugin>rokae_ros2_control/RokaeHardware</plugin>
-                <param name="arm_ip">192.168.2.160</param>
-<!--                <param name="joint_impedance">500,500,500,500,50,50,50</param>-->
-                <param name="local_ip">192.168.2.233</param>
-            </hardware>
-            <xacro:ar5_interfaces name="left"/>
-            <xacro:if value="${'$(arg type)' == 'rg75'}">
-                <joint name="left_gripper_joint">
-                    <command_interface name="position"/>
-                    <state_interface name="position">
-                        <param name="initial_value">0</param>
-                    </state_interface>
-                </joint>
-            </xacro:if>
-        </ros2_control>
-        <ros2_control name="ar5_right_system" type="system">
-            <hardware>
-                <plugin>rokae_ros2_control/RokaeHardware</plugin>
-                <param name="arm_ip">192.168.2.161</param>
-                <param name="joint_impedance">500,500,500,500,50,50,50</param>
-                <param name="local_ip">192.168.2.233</param>
-            </hardware>
-            <xacro:ar5_interfaces name="right"/>
-            <xacro:if value="${'$(arg type)' == 'rg75'}">
-                <joint name="right_gripper_joint">
-                    <command_interface name="position"/>
-                    <state_interface name="position">
-                        <param name="initial_value">0</param>
-                    </state_interface>
-                </joint>
-            </xacro:if>
-        </ros2_control>
-        <ros2_control name="eyou_body" type="system">
-            <hardware>
-                <plugin>eyou_ros2_control/EyouHardware</plugin>
-                <param name="device_type">Canable</param>
-                <param name="device_index">0</param>
-                <param name="baudrate">1000</param>
-                <param name="motor_ids">[1, 2, 3, 4, 5, 6]</param>
-                <param name="control_period_ms">4</param>
-                <param name="report_period_ms">100</param>
-                <param name="use_sync">true</param>
-                <!-- 每个电机的减速比配置 -->
-                <param name="reduction_ratios">[121.0, 121.0, 121.0, 121.0, 56.0, 36.0]</param>
-            </hardware>
-            <xacro:body_interfaces/>
-        </ros2_control>
-        <ros2_control name="virtual_system" type="system">
-            <hardware>
-                <plugin>mock_components/GenericSystem</plugin>
-            </hardware>
-            <xacro:chassis_interfaces/>
-        </ros2_control>
-    </xacro:if>
-    <xacro:unless value="${'$(arg ros2_control_hardware_type)' == 'real'}">
-        <xacro:unless value="${'$(arg ros2_control_hardware_type)' == 'real-laptop'}">
-        <ros2_control name="fiveages_w1_system" type="system">
-            <hardware>
-                <xacro:if value="${'$(arg ros2_control_hardware_type)' == 'gz'}">
-                    <plugin>gz_ros2_control/GazeboSimSystem</plugin>
-                </xacro:if>
-                <xacro:if value="${'$(arg ros2_control_hardware_type)' == 'mock_components'}">
-                    <plugin>mock_components/GenericSystem</plugin>
-                </xacro:if>
-                <xacro:if value="${'$(arg ros2_control_hardware_type)' == 'isaac'}">
-                    <plugin>topic_based_ros2_control/TopicBasedSystem</plugin>
-                    <param name="joint_commands_topic">/isaac/joint_command</param>
-                    <param name="joint_states_topic">/isaac/joint_states</param>
-                    <param name="sum_wrapped_joint_states">false</param>
-                    <param name="initialize_commands_from_state">true</param>
-                </xacro:if>
-            </hardware>
-            <xacro:chassis_interfaces/>
-            <xacro:body_interfaces/>
-            <xacro:ar5_interfaces name="left"/>
-            <xacro:ar5_interfaces name="right"/>
-            <xacro:if value="${'$(arg type)' == 'rg75' or '$(arg type)' == 'leapmotor' or '$(arg type)' == 'linkhou_rg75' or '$(arg type)' == 'linkhou_leapmotor'}">
-                <xacro:include filename="$(find jodell_description)/xacro/ros2_control/RG75-300.xacro"/>
-                <xacro:rg75_interfaces name="left"/>
-                <xacro:rg75_interfaces name="right"/>
-            </xacro:if>
-        </ros2_control>
-        </xacro:unless>
-    </xacro:unless>
-    <!-- Gazebo plugin configuration -->
-    <xacro:arg name="gazebo" default="false"/>
-    <xacro:if value="$(arg gazebo)">
-        <xacro:property name="ros2_control_config_basename" value="ros2_controllers.yaml"/>
-        <xacro:if value="${type_arg == 'rg75'}">
-            <xacro:property name="ros2_control_config_basename" value="rg75.yaml"/>
-        </xacro:if>
-        <xacro:if value="${type_arg == 'leapmotor'}">
-            <xacro:property name="ros2_control_config_basename" value="leapmotor.yaml"/>
-        </xacro:if>
-        <xacro:if value="${type_arg == 'linkhou_rg75'}">
-            <xacro:property name="ros2_control_config_basename" value="linkhou_rg75.yaml"/>
-        </xacro:if>
-        <xacro:if value="${type_arg == 'linkhou_leapmotor'}">
-            <xacro:property name="ros2_control_config_basename" value="linkhou_leapmotor.yaml"/>
-        </xacro:if>
-        <gazebo>
-            <plugin filename="gz_ros2_control-system" name="gz_ros2_control::GazeboSimROS2ControlPlugin">
-                <parameters>$(find fiveages_w1_description)/config/ros2_control/${ros2_control_config_basename}</parameters>
-            </plugin>
-        </gazebo>
-        <xacro:include filename="$(find fiveages_w1_description)/xacro/gazebo.xacro"/>
-    </xacro:if>
+	<xacro:arg name="ros2_control_hardware_type" default="mock_components"/>
+	<!-- 直接include robot.xacro并根据type参数传递 -->
+	<xacro:include filename="$(find fiveages_w1_description)/xacro/robot.xacro"/>
+	<xacro:include filename="$(find rokae_ar5_description)/xacro/ros2_control/interfaces.xacro"/>
+	<xacro:include filename="$(find fiveages_w1_description)/xacro/ros2_control/body.xacro"/>
+	<xacro:include filename="$(find fiveages_w1_description)/xacro/ros2_control/chassis.xacro"/>
+	<xacro:if value="${'$(arg ros2_control_hardware_type)' == 'real'}">
+		<ros2_control name="ar5_left_system" type="system">
+			<hardware>
+				<plugin>rokae_ros2_control/RokaeHardware</plugin>
+				<param name="arm_ip">192.168.2.160</param>
+				<param name="joint_impedance">500,500,500,500,50,50,50</param>
+				<param name="local_ip">192.168.2.100</param>
+			</hardware>
+			<xacro:ar5_interfaces name="left"/>
+			<xacro:if value="${'$(arg type)' == 'rg75'}">
+				<joint name="left_gripper_joint">
+					<command_interface name="position"/>
+					<state_interface name="position">
+						<param name="initial_value">0</param>
+					</state_interface>
+				</joint>
+			</xacro:if>
+		</ros2_control>
+		<ros2_control name="ar5_right_system" type="system">
+			<hardware>
+				<plugin>rokae_ros2_control/RokaeHardware</plugin>
+				<param name="arm_ip">192.168.2.161</param>
+				<param name="joint_impedance">500,500,500,500,50,50,50</param>
+				<param name="local_ip">192.168.2.100</param>
+			</hardware>
+			<xacro:ar5_interfaces name="right"/>
+			<xacro:if value="${'$(arg type)' == 'rg75'}">
+				<joint name="right_gripper_joint">
+					<command_interface name="position"/>
+					<state_interface name="position">
+						<param name="initial_value">0</param>
+					</state_interface>
+				</joint>
+			</xacro:if>
+		</ros2_control>
+		<ros2_control name="eyou_body" type="system">
+			<hardware>
+				<plugin>eyou_ros2_control/EyouHardware</plugin>
+				<param name="device_type">Canable</param>
+				<param name="device_index">2</param>
+				<param name="baudrate">1000</param>
+				<param name="motor_ids">[1, 2, 3, 4, 5, 6]</param>
+				<param name="control_period_ms">4</param>
+				<param name="report_period_ms">100</param>
+				<param name="use_sync">true</param>
+				<!-- 每个电机的减速比配置 -->
+				<param name="reduction_ratios">[121.0, 121.0, 121.0, 121.0, 56.0, 36.0]</param>
+			</hardware>
+			<xacro:body_interfaces/>
+		</ros2_control>
+		<ros2_control name="virtual_system" type="system">
+			<hardware>
+				<plugin>mock_components/GenericSystem</plugin>
+			</hardware>
+			<xacro:chassis_interfaces/>
+		</ros2_control>
+	</xacro:if>
+	<xacro:if value="${'$(arg ros2_control_hardware_type)' == 'real-laptop'}">
+		<ros2_control name="ar5_left_system" type="system">
+			<hardware>
+				<plugin>rokae_ros2_control/RokaeHardware</plugin>
+				<param name="arm_ip">192.168.2.160</param>
+				<!--                <param name="joint_impedance">500,500,500,500,50,50,50</param>-->
+				<param name="local_ip">192.168.2.233</param>
+			</hardware>
+			<xacro:ar5_interfaces name="left"/>
+			<xacro:if value="${'$(arg type)' == 'rg75'}">
+				<joint name="left_gripper_joint">
+					<command_interface name="position"/>
+					<state_interface name="position">
+						<param name="initial_value">0</param>
+					</state_interface>
+				</joint>
+			</xacro:if>
+		</ros2_control>
+		<ros2_control name="ar5_right_system" type="system">
+			<hardware>
+				<plugin>rokae_ros2_control/RokaeHardware</plugin>
+				<param name="arm_ip">192.168.2.161</param>
+				<param name="joint_impedance">500,500,500,500,50,50,50</param>
+				<param name="local_ip">192.168.2.233</param>
+			</hardware>
+			<xacro:ar5_interfaces name="right"/>
+			<xacro:if value="${'$(arg type)' == 'rg75'}">
+				<joint name="right_gripper_joint">
+					<command_interface name="position"/>
+					<state_interface name="position">
+						<param name="initial_value">0</param>
+					</state_interface>
+				</joint>
+			</xacro:if>
+		</ros2_control>
+		<ros2_control name="eyou_body" type="system">
+			<hardware>
+				<plugin>eyou_ros2_control/EyouHardware</plugin>
+				<param name="device_type">Canable</param>
+				<param name="device_index">0</param>
+				<param name="baudrate">1000</param>
+				<param name="motor_ids">[1, 2, 3, 4, 5, 6]</param>
+				<param name="control_period_ms">4</param>
+				<param name="report_period_ms">100</param>
+				<param name="use_sync">true</param>
+				<!-- 每个电机的减速比配置 -->
+				<param name="reduction_ratios">[121.0, 121.0, 121.0, 121.0, 56.0, 36.0]</param>
+			</hardware>
+			<xacro:body_interfaces/>
+		</ros2_control>
+		<ros2_control name="virtual_system" type="system">
+			<hardware>
+				<plugin>mock_components/GenericSystem</plugin>
+			</hardware>
+			<xacro:chassis_interfaces/>
+		</ros2_control>
+	</xacro:if>
+	<xacro:unless value="${'$(arg ros2_control_hardware_type)' == 'real'}">
+		<xacro:unless value="${'$(arg ros2_control_hardware_type)' == 'real-laptop'}">
+			<ros2_control name="fiveages_w1_system" type="system">
+				<hardware>
+					<xacro:if value="${'$(arg ros2_control_hardware_type)' == 'gz'}">
+						<plugin>gz_ros2_control/GazeboSimSystem</plugin>
+					</xacro:if>
+					<xacro:if value="${'$(arg ros2_control_hardware_type)' == 'mock_components'}">
+						<plugin>mock_components/GenericSystem</plugin>
+					</xacro:if>
+					<xacro:if value="${'$(arg ros2_control_hardware_type)' == 'isaac'}">
+						<plugin>topic_based_ros2_control/TopicBasedSystem</plugin>
+						<param name="joint_commands_topic">/isaac/joint_command</param>
+						<param name="joint_states_topic">/isaac/joint_states</param>
+						<param name="sum_wrapped_joint_states">false</param>
+						<param name="initialize_commands_from_state">true</param>
+					</xacro:if>
+				</hardware>
+				<xacro:unless value="${'$(arg ros2_control_hardware_type)' == 'isaac'}">
+					<xacro:chassis_interfaces/>
+				</xacro:unless>
+				<xacro:body_interfaces/>
+				<xacro:ar5_interfaces name="left"/>
+				<xacro:ar5_interfaces name="right"/>
+				<xacro:if
+						value="${'$(arg type)' == 'rg75' or '$(arg type)' == 'leapmotor' or '$(arg type)' == 'linkhou_rg75' or '$(arg type)' == 'linkhou_leapmotor'}">
+					<xacro:include filename="$(find jodell_description)/xacro/ros2_control/RG75-300.xacro"/>
+					<xacro:rg75_interfaces name="left"/>
+					<xacro:rg75_interfaces name="right"/>
+				</xacro:if>
+			</ros2_control>
+		</xacro:unless>
+	</xacro:unless>
+	<!-- Gazebo plugin configuration -->
+	<xacro:arg name="gazebo" default="false"/>
+	<xacro:if value="$(arg gazebo)">
+		<xacro:property name="ros2_control_config_basename" value="ros2_controllers.yaml"/>
+		<xacro:if value="${type_arg == 'rg75'}">
+			<xacro:property name="ros2_control_config_basename" value="rg75.yaml"/>
+		</xacro:if>
+		<xacro:if value="${type_arg == 'leapmotor'}">
+			<xacro:property name="ros2_control_config_basename" value="leapmotor.yaml"/>
+		</xacro:if>
+		<xacro:if value="${type_arg == 'linkhou_rg75'}">
+			<xacro:property name="ros2_control_config_basename" value="linkhou_rg75.yaml"/>
+		</xacro:if>
+		<xacro:if value="${type_arg == 'linkhou_leapmotor'}">
+			<xacro:property name="ros2_control_config_basename" value="linkhou_leapmotor.yaml"/>
+		</xacro:if>
+		<gazebo>
+			<plugin filename="gz_ros2_control-system" name="gz_ros2_control::GazeboSimROS2ControlPlugin">
+				<parameters>$(find fiveages_w1_description)/config/ros2_control/${ros2_control_config_basename}</parameters>
+			</plugin>
+		</gazebo>
+		<xacro:include filename="$(find fiveages_w1_description)/xacro/gazebo.xacro"/>
+	</xacro:if>
 </robot>
