Commit message: Add jodell-rg75 and leapmotor gripper configurations

File: xacro/grippers.xacro (robot description, xacro)
@@ -42,4 +42,32 @@
 			</joint>
 		</xacro:if>
+		<xacro:if value="${'$(arg type)' == 'jodell-rg75'}">
+			<xacro:include filename="$(find jodell_description)/xacro/RG75-300.xacro"/>
+			<xacro:RG75-300 name="left" use_flange="true"/>
+			<xacro:RG75-300 name="right" use_flange="true"/>
+			<joint name="left_gripper_base_joint" type="fixed">
+				<parent link="left_link7"/>
+				<child link="left_flange"/>
+			</joint>
+			<joint name="right_gripper_base_joint" type="fixed">
+				<origin xyz="0 0 -0.0045"/>
+				<parent link="right_link7"/>
+				<child link="right_flange"/>
+			</joint>
+		</xacro:if>
+		<xacro:if value="${'$(arg type)' == 'leapmotor'}">
+			<xacro:include filename="$(find jodell_description)/xacro/RG75-300.xacro"/>
+			<xacro:RG75-300 name="left" use_flange="true" pad="leapmotor"/>
+			<xacro:RG75-300 name="right" use_flange="true" pad="leapmotor"/>
+			<joint name="left_gripper_base_joint" type="fixed">
+				<parent link="left_link7"/>
+				<child link="left_flange"/>
+			</joint>
+			<joint name="right_gripper_base_joint" type="fixed">
+				<origin xyz="0 0 -0.0045"/>
+				<parent link="right_link7"/>
+				<child link="right_flange"/>
+			</joint>
+		</xacro:if>
 	</xacro:macro>
 </robot>

Commit message: isaac sim simulation

File: xacro/grippers.xacro (robot description, xacro)
@@ -47,4 +47,5 @@
             <xacro:RG75-300 name="right" use_flange="true"/>
             <joint name="left_gripper_base_joint" type="fixed">
+                <origin xyz="0 0 -0.0045"/>
                 <parent link="left_link7"/>
                 <child link="left_flange"/>

File: xacro/ros2_control/chassis.xacro (robot description, xacro)
@@ -1,23 +1,26 @@
 <?xml version="1.0"?>
 <robot xmlns:xacro="http://www.ros.org/wiki/xacro">
-  <xacro:macro name="chassis_interfaces">
-    <joint name="chassis_left_joint">
-      <command_interface name="velocity">
-        <param name="min">-1.0</param>
-        <param name="max">1.0</param>
-      </command_interface>
-      <state_interface name="position"/>
-      <state_interface name="velocity"/>
-      <state_interface name="effort"/>
-    </joint>
-    <joint name="chassis_right_joint">
-      <command_interface name="velocity">
-        <param name="min">-1.0</param>
-        <param name="max">1.0</param>
-      </command_interface>
-      <state_interface name="position"/>
-      <state_interface name="velocity"/>
-      <state_interface name="effort"/>
-    </joint>
-  </xacro:macro>
+    <xacro:macro name="chassis_interfaces">
+        <xacro:arg name="gazebo" default="false"/>
+        <xacro:if value="$(arg gazebo)">
+            <joint name="chassis_left_joint">
+                <command_interface name="velocity">
+                    <param name="min">-1.0</param>
+                    <param name="max">1.0</param>
+                </command_interface>
+                <state_interface name="position"/>
+                <state_interface name="velocity"/>
+                <state_interface name="effort"/>
+            </joint>
+            <joint name="chassis_right_joint">
+                <command_interface name="velocity">
+                    <param name="min">-1.0</param>
+                    <param name="max">1.0</param>
+                </command_interface>
+                <state_interface name="position"/>
+                <state_interface name="velocity"/>
+                <state_interface name="effort"/>
+            </joint>
+        </xacro:if>
+    </xacro:macro>
 </robot>

Commit message: 修改了type相关 在type里同时写chassis和gripper

File: xacro/grippers.xacro (robot description, xacro)
@@ -1,7 +1,7 @@
 <?xml version="1.0"?>
 <robot xmlns:xacro="http://www.ros.org/wiki/xacro">
-    <xacro:macro name="Grippers">
-        <xacro:arg name="type" default="empty"/>
-        <xacro:if value="${'$(arg type)' == 'robotiq85'}">
+    <xacro:macro name="Grippers" params="type:=''">
+        <!-- Note: type parameter is now passed as macro parameter -->
+        <xacro:if value="${type == 'robotiq85'}">
             <xacro:include filename="$(find robotiq_description)/xacro/2F85.xacro"/>
             <xacro:Robotiq85 name="left"/>
@@ -16,5 +16,5 @@
             </joint>
         </xacro:if>
-        <xacro:if value="${'$(arg type)' == 'AG2F90-C'}">
+        <xacro:if value="${type == 'AG2F90-C'}">
             <xacro:include filename="$(find changingtek_description)/xacro/AG2F90-C.xacro"/>
             <xacro:AG2F90-C name="left"/>
@@ -29,5 +29,5 @@
             </joint>
         </xacro:if>
-        <xacro:if value="${'$(arg type)' == 'AG2F120S'}">
+        <xacro:if value="${type == 'AG2F120S'}">
             <xacro:include filename="$(find changingtek_description)/xacro/AG2F120S.xacro"/>
             <xacro:AG2F120S name="left"/>
@@ -42,5 +42,5 @@
             </joint>
         </xacro:if>
-        <xacro:if value="${'$(arg type)' == 'rg75'}">
+        <xacro:if value="${type == 'rg75'}">
             <xacro:include filename="$(find jodell_description)/xacro/RG75-300.xacro"/>
             <xacro:RG75-300 name="left" use_flange="true"/>
@@ -57,9 +57,10 @@
             </joint>
         </xacro:if>
-        <xacro:if value="${'$(arg type)' == 'leapmotor'}">
+        <xacro:if value="${type == 'leapmotor'}">
             <xacro:include filename="$(find jodell_description)/xacro/RG75-300.xacro"/>
             <xacro:RG75-300 name="left" use_flange="true" pad="leapmotor"/>
             <xacro:RG75-300 name="right" use_flange="true" pad="leapmotor"/>
             <joint name="left_gripper_base_joint" type="fixed">
+                <origin xyz="0 0 -0.0045"/>
                 <parent link="left_link7"/>
                 <child link="left_flange"/>

File: xacro/robot.xacro (robot description, xacro)
@@ -2,7 +2,15 @@
 <robot name="FiveAges W1" xmlns:xacro="http://www.ros.org/wiki/xacro">
 	<!-- Arguments -->
-	<xacro:arg name="chassis" default="chassis"/>
+	<xacro:arg name="type" default=""/>
+	<!-- Select chassis & gripper based on type -->
+	<xacro:property name="type_arg" value="$(arg type)"/>
+	<xacro:property name="selected_chassis" value="chassis"/>
+	<xacro:property name="selected_gripper_type" value="${type_arg}"/>
+	<xacro:if value="${type_arg == 'linkhou_rg75'}">
+		<xacro:property name="selected_chassis" value="linkhou_q1"/>
+		<xacro:property name="selected_gripper_type" value="rg75"/>
+	</xacro:if>
 	<!-- Include Component Macros -->
-	<xacro:include filename="$(find fiveages_w1_description)/xacro/chassis/$(arg chassis).xacro"/>
+	<xacro:include filename="$(find fiveages_w1_description)/xacro/chassis/${selected_chassis}.xacro"/>
 	<xacro:include filename="$(find fiveages_w1_description)/xacro/body.xacro"/>
 	<xacro:include filename="$(find rokae_ar5_description)/xacro/arm.xacro"/>
@@ -25,4 +33,4 @@
 	<xacro:Arm name="left" direction="1"/>
 	<xacro:Arm name="right" direction="-1"/>
-	<xacro:Grippers/>
+	<xacro:Grippers type="${selected_gripper_type}"/>
 </robot>
