Commit message: add fiveages mesh

File: xacro/body.xacro (robot description, xacro)
@@ -182,5 +182,5 @@
 		</link>
 		<joint name="head_joint1" type="revolute">
-			<origin xyz="-0.026 0 0.487"/>
+			<origin xyz="-0.02258 0 0.485317"/>
 			<parent link="body_link4"/>
 			<child link="head_link1"/>
@@ -213,5 +213,5 @@
 		</link>
 		<joint name="head_joint2" type="revolute">
-			<origin xyz="0 0.0243 0.041"/>
+			<origin xyz="0 0 0.033543"/>
 			<parent link="head_link1"/>
 			<child link="head_link2"/>

Commit message: simplified mesh for fa 1

File: xacro/body.xacro (robot description, xacro)
@@ -15,14 +15,4 @@
                         izz="0.014637715325779"/>
             </inertial>
-            <visual>
-                <geometry>
-                    <mesh filename="file://$(find fiveages_w1_description)/meshes/body/base.obj"/>
-                </geometry>
-            </visual>
-            <collision>
-                <geometry>
-                    <mesh filename="file://$(find fiveages_w1_description)/meshes/body/base.obj"/>
-                </geometry>
-            </collision>
         </link>
         <!-- Trunk Base Joint -->

Commit message: ADD self collision config for rokae ar5 dual

File: xacro/body.xacro (robot description, xacro)
@@ -1,5 +1,5 @@
 <?xml version="1.0"?>
 <robot xmlns:xacro="http://www.ros.org/wiki/xacro">
-    <xacro:macro name="Body">
+    <xacro:macro name="Body" params="collider:=convex">
         <!-- Trunk Base Link -->
         <link name="trunk_base_link">
@@ -15,4 +15,11 @@
                         izz="0.014637715325779"/>
             </inertial>
+            <xacro:if value="${collider == 'convex'}">
+                <collision>
+                    <geometry>
+                        <mesh filename="file://$(find fiveages_w1_description)/meshes/body/base.obj"/>
+                    </geometry>
+                </collision>
+            </xacro:if>
         </link>
         <!-- Trunk Base Joint -->
@@ -41,9 +48,11 @@
                 </geometry>
             </visual>
-            <collision>
-                <geometry>
-                    <mesh filename="file://$(find fiveages_w1_description)/meshes/body/link1.obj"/>
-                </geometry>
-            </collision>
+            <xacro:if value="${collider == 'convex'}">
+                <collision>
+                    <geometry>
+                        <mesh filename="file://$(find fiveages_w1_description)/meshes/body/link1.obj"/>
+                    </geometry>
+                </collision>
+            </xacro:if>
         </link>
         <joint name="body_joint1" type="revolute">
@@ -72,9 +81,11 @@
                 </geometry>
             </visual>
-            <collision>
-                <geometry>
-                    <mesh filename="file://$(find fiveages_w1_description)/meshes/body/link2.obj"/>
-                </geometry>
-            </collision>
+            <xacro:if value="${collider == 'convex'}">
+                <collision>
+                    <geometry>
+                        <mesh filename="file://$(find fiveages_w1_description)/meshes/body/link2.obj"/>
+                    </geometry>
+                </collision>
+            </xacro:if>
         </link>
         <joint name="body_joint2" type="revolute">
@@ -103,9 +114,11 @@
                 </geometry>
             </visual>
-            <collision>
-                <geometry>
-                    <mesh filename="file://$(find fiveages_w1_description)/meshes/body/link3.obj"/>
-                </geometry>
-            </collision>
+            <xacro:if value="${collider == 'convex'}">
+                <collision>
+                    <geometry>
+                        <mesh filename="file://$(find fiveages_w1_description)/meshes/body/link3.obj"/>
+                    </geometry>
+                </collision>
+            </xacro:if>
         </link>
         <joint name="body_joint3" type="revolute">
@@ -134,9 +147,19 @@
                 </geometry>
             </visual>
-            <collision>
-                <geometry>
-                    <mesh filename="file://$(find fiveages_w1_description)/meshes/body/link4.obj"/>
-                </geometry>
-            </collision>
+            <xacro:if value="${collider == 'convex'}">
+                <collision>
+                    <geometry>
+                        <mesh filename="file://$(find fiveages_w1_description)/meshes/body/link4.obj"/>
+                    </geometry>
+                </collision>
+            </xacro:if>
+            <xacro:if value="${collider == 'simple'}">
+                <collision>
+                    <origin xyz="0.0091 0 0.256"/>
+                    <geometry>
+                        <box size="0.2509 0.35 0.5029"/>
+                    </geometry>
+                </collision>
+            </xacro:if>
         </link>
         <joint name="body_joint4" type="revolute">
@@ -165,9 +188,19 @@
                 </geometry>
             </visual>
-            <collision>
-                <geometry>
-                    <mesh filename="file://$(find fiveages_w1_description)/meshes/body/head1.obj"/>
-                </geometry>
-            </collision>
+            <xacro:if value="${collider == 'convex'}">
+                <collision>
+                    <geometry>
+                        <mesh filename="file://$(find fiveages_w1_description)/meshes/body/head1.obj"/>
+                    </geometry>
+                </collision>
+            </xacro:if>
+            <xacro:if value="${collider == 'simple'}">
+                <collision>
+                    <origin xyz="0.0003 0.0000 -0.0100"/>
+                    <geometry>
+                        <box size="0.0500 0.0500 0.0401"/>
+                    </geometry>
+                </collision>
+            </xacro:if>
         </link>
         <joint name="head_joint1" type="revolute">
@@ -181,5 +214,5 @@
         <link name="head_link2">
             <inertial>
-                <origin xyz="1.3878E-16 -0.0243 0.093841"/>
+                <origin xyz="0.02 0 0.093841"/>
                 <mass value="1.2686"/>
                 <inertia
@@ -196,9 +229,19 @@
                 </geometry>
             </visual>
-            <collision>
-                <geometry>
-                    <mesh filename="file://$(find fiveages_w1_description)/meshes/body/head2.obj"/>
-                </geometry>
-            </collision>
+            <xacro:if value="${collider == 'convex'}">
+                <collision>
+                    <geometry>
+                        <mesh filename="file://$(find fiveages_w1_description)/meshes/body/head2.obj"/>
+                    </geometry>
+                </collision>
+            </xacro:if>
+            <xacro:if value="${collider == 'simple'}">
+                <collision>
+                    <origin xyz="0.0366 0 0.08"/>
+                    <geometry>
+                        <box size="0.1813 0.1640 0.2230"/>
+                    </geometry>
+                </collision>
+            </xacro:if>
         </link>
         <joint name="head_joint2" type="revolute">

File: xacro/robot.xacro (robot description, xacro)
@@ -3,4 +3,5 @@
 	<!-- Arguments -->
 	<xacro:arg name="type" default=""/>
+	<xacro:arg name="collider" default="convex"/>
 	<!-- Select chassis & gripper based on type -->
 	<xacro:property name="type_arg" value="$(arg type)"/>
@@ -23,5 +24,5 @@
 	<xacro:Chassis/>
 	<!-- Body -->
-	<xacro:Body/>
+	<xacro:Body collider="$(arg collider)"/>
 	<link name="arm_base"/>
 	<joint name="arm_base_joint" type="fixed">
@@ -41,6 +42,6 @@
 	</joint>
 	<!-- Arms -->
-	<xacro:Arm name="left" direction="1"/>
-	<xacro:Arm name="right" direction="-1"/>
+	<xacro:Arm name="left" collider="$(arg collider)" direction="1"/>
+	<xacro:Arm name="right" collider="$(arg collider)" direction="-1"/>
 	<xacro:Grippers type="${selected_gripper_type}"/>
 </robot>

Commit message: upper body component

File: xacro/body.xacro (robot description, xacro)
@@ -253,4 +253,10 @@
             <dynamics damping="0.01" friction="0.1"/>
         </joint>
+        <link name="arm_base"/>
+        <joint name="arm_base_joint" type="fixed">
+            <parent link="body_link4"/>
+            <child link="arm_base"/>
+            <origin xyz="0.0 0.0 0.41"/>
+        </joint>
     </xacro:macro>
 </robot>

File: xacro/component.xacro (robot description, xacro)
@@ -16,21 +16,6 @@
 	<xacro:if value="${'$(arg type)' == 'upper_body'}">
 		<xacro:include filename="$(find fiveages_w1_description)/xacro/body.xacro"/>
-		<xacro:include filename="$(find rokae_ar5_description)/xacro/arm.xacro"/>
 		<link name="base_link"/>
-		<!-- Body -->
 		<xacro:Body/>
-		<joint name="left_arm_mount" type="fixed">
-			<parent link="body_link4"/>
-			<child link="left_base_link"/>
-			<origin xyz="0.0 0.12 0.41" rpy="-1.57 1.57 0"/>
-		</joint>
-		<joint name="right_arm_mount" type="fixed">
-			<parent link="body_link4"/>
-			<child link="right_base_link"/>
-			<origin xyz="0.0 -0.12 0.41" rpy="1.57 1.57 0"/>
-		</joint>
-		<!-- Arms -->
-		<xacro:Arm name="left" direction="1"/>
-		<xacro:Arm name="right" direction="-1"/>
 	</xacro:if>
 </robot>

File: xacro/robot.xacro (robot description, xacro)
@@ -25,10 +25,4 @@
 	<!-- Body -->
 	<xacro:Body collider="$(arg collider)"/>
-	<link name="arm_base"/>
-	<joint name="arm_base_joint" type="fixed">
-		<parent link="body_link4"/>
-		<child link="arm_base"/>
-		<origin xyz="0.0 0.0 0.41"/>
-	</joint>
 	<joint name="left_arm_mount" type="fixed">
 		<parent link="arm_base"/>
