Commit message: update rokae ros2 control

File: xacro/body.xacro (robot description, xacro)
@@ -1,4 +1,22 @@
 <?xml version="1.0"?>
 <robot xmlns:xacro="http://www.ros.org/wiki/xacro">
+    <!-- Shared by full Body and topology:=dual planning URDF. -->
+    <xacro:macro name="body_link4_collision" params="collider">
+        <xacro:if value="${collider == 'convex'}">
+            <collision>
+                <geometry>
+                    <mesh filename="file://$(find fiveages_w1_description)/meshes/body/link4.glb"/>
+                </geometry>
+            </collision>
+        </xacro:if>
+        <xacro:if value="${collider == 'simple'}">
+            <collision>
+                <origin xyz="0.0091 0 0.256"/>
+                <geometry>
+                    <box size="0.2509 0.35 0.5029"/>
+                </geometry>
+            </collision>
+        </xacro:if>
+    </xacro:macro>
     <xacro:macro name="Body" params="collider:=convex">
         <!-- Trunk Base Link -->
@@ -147,19 +165,5 @@
                 </geometry>
             </visual>
-            <xacro:if value="${collider == 'convex'}">
-                <collision>
-                    <geometry>
-                        <mesh filename="file://$(find fiveages_w1_description)/meshes/body/link4.glb"/>
-                    </geometry>
-                </collision>
-            </xacro:if>
-            <xacro:if value="${collider == 'simple'}">
-                <collision>
-                    <origin xyz="0.0091 0 0.256"/>
-                    <geometry>
-                        <box size="0.2509 0.35 0.5029"/>
-                    </geometry>
-                </collision>
-            </xacro:if>
+            <xacro:body_link4_collision collider="${collider}"/>
         </link>
         <joint name="body_joint4" type="revolute">

File: xacro/robot.xacro (robot description, xacro)
@@ -2,5 +2,11 @@
 <robot name="FiveAges W1" xmlns:xacro="http://www.ros.org/wiki/xacro">
     <xacro:property name="PI" value="3.1415926535897931"/>
-    <xacro:arg name="collider" default="convex"/>
+    <!-- topology:
+         full (default) = chassis + body/head + dual AR5
+         dual           = split_body planning URDF (same layout as m6_ccs / WCE3):
+                          empty base_link is the URDF root; arm_base is OCS2 baseFrame
+                          and carries the W1 chest box. Flange ±0.12. -->
+    <xacro:arg name="topology" default="full"/>
+    <xacro:arg name="collider" default="simple"/>
     <!-- Native W1 chassis, or Linkhou Q1. Independent from the dual-arm kit. -->
     <xacro:arg name="chassis" default="w1"/>
@@ -21,4 +27,5 @@
     <xacro:arg name="right_tcp_offset_xyz" default="0 0 0"/>
     <xacro:arg name="right_tcp_offset_rpy" default="0 0 0"/>
+    <xacro:property name="topology_arg" value="$(arg topology)"/>
     <xacro:property name="type_arg" value="$(arg type)"/>
     <xacro:property name="left_type_arg" value="$(arg left_type)"/>
@@ -32,25 +39,55 @@
     <xacro:property name="selected_gripper_type" value="${left_gripper_type if left_gripper_type == right_gripper_type else ''}"/>
     <xacro:property name="selected_gripper_pad" value="${left_gripper_pad if left_gripper_pad == right_gripper_pad else 'default'}"/>
-    <xacro:property name="chassis_arg" value="$(arg chassis)"/>
-    <xacro:if value="${chassis_arg == 'w1'}">
-        <xacro:include filename="$(find fiveages_w1_description)/xacro/chassis/chassis.xacro"/>
-        <xacro:Chassis joints_movable="$(arg chassis_joints_movable)"/>
+    <!-- CCS and SRS share the W1 flange (±0.12), not the CCS pedestal ±0.062. -->
+    <xacro:if value="${topology_arg == 'dual'}">
+        <link name="base_link"/>
+        <!-- body_link4 simple box (origin 0.0091 0 0.256, size 0.2509 0.35 0.5029)
+             expressed in arm_base (body_link4 → arm_base z=+0.41). -->
+        <link name="arm_base">
+            <collision>
+                <origin xyz="0.0091 0 -0.154"/>
+                <geometry>
+                    <box size="0.2509 0.35 0.5029"/>
+                </geometry>
+            </collision>
+        </link>
+        <joint name="arm_base_joint" type="fixed">
+            <parent link="base_link"/>
+            <child link="arm_base"/>
+        </joint>
+        <joint name="left_arm_mount" type="fixed">
+            <parent link="arm_base"/>
+            <child link="left_base_link"/>
+            <origin xyz="0.0 0.12 0" rpy="-${PI/2} ${PI/2} 0"/>
+        </joint>
+        <joint name="right_arm_mount" type="fixed">
+            <parent link="arm_base"/>
+            <child link="right_base_link"/>
+            <origin xyz="0.0 -0.12 0" rpy="${PI/2} ${PI/2} 0"/>
+        </joint>
     </xacro:if>
-    <xacro:if value="${chassis_arg == 'linkhou_q1'}">
-        <xacro:include filename="$(find fiveages_w1_description)/xacro/chassis/linkhou_q1.xacro"/>
-        <xacro:Chassis joints_movable="$(arg chassis_joints_movable)"/>
-    </xacro:if>
-    <xacro:include filename="$(find fiveages_w1_description)/xacro/body.xacro"/>
-    <xacro:Body collider="$(arg collider)"/>
-    <joint name="left_arm_mount" type="fixed">
-        <parent link="arm_base"/>
-        <child link="left_base_link"/>
-        <origin xyz="0.0 0.12 0" rpy="-${PI/2} ${PI/2} 0"/>
-    </joint>
-    <joint name="right_arm_mount" type="fixed">
-        <parent link="arm_base"/>
-        <child link="right_base_link"/>
-        <origin xyz="0.0 -0.12 0" rpy="${PI/2} ${PI/2} 0"/>
-    </joint>
+    <xacro:unless value="${topology_arg == 'dual'}">
+        <xacro:property name="chassis_arg" value="$(arg chassis)"/>
+        <xacro:if value="${chassis_arg == 'w1'}">
+            <xacro:include filename="$(find fiveages_w1_description)/xacro/chassis/chassis.xacro"/>
+            <xacro:Chassis joints_movable="$(arg chassis_joints_movable)"/>
+        </xacro:if>
+        <xacro:if value="${chassis_arg == 'linkhou_q1'}">
+            <xacro:include filename="$(find fiveages_w1_description)/xacro/chassis/linkhou_q1.xacro"/>
+            <xacro:Chassis joints_movable="$(arg chassis_joints_movable)"/>
+        </xacro:if>
+        <xacro:include filename="$(find fiveages_w1_description)/xacro/body.xacro"/>
+        <xacro:Body collider="$(arg collider)"/>
+        <joint name="left_arm_mount" type="fixed">
+            <parent link="arm_base"/>
+            <child link="left_base_link"/>
+            <origin xyz="0.0 0.12 0" rpy="-${PI/2} ${PI/2} 0"/>
+        </joint>
+        <joint name="right_arm_mount" type="fixed">
+            <parent link="arm_base"/>
+            <child link="right_base_link"/>
+            <origin xyz="0.0 -0.12 0" rpy="${PI/2} ${PI/2} 0"/>
+        </joint>
+    </xacro:unless>
     <xacro:if value="${'$(arg arms)' == 'ar5_ccs'}">
         <xacro:include filename="$(find ar5_ccs_description)/xacro/arm_ccs.xacro"/>

Commit message: w1 refactor

File: xacro/body.xacro (robot description, xacro)
@@ -33,4 +33,9 @@
                         izz="0.014637715325779"/>
             </inertial>
+            <visual>
+                <geometry>
+                    <mesh filename="file://$(find fiveages_w1_description)/meshes/body/base.glb"/>
+                </geometry>
+            </visual>
             <xacro:if value="${collider == 'convex'}">
                 <collision>

File: xacro/chassis/chassis.xacro (robot description, xacro)
@@ -4,5 +4,5 @@
     <xacro:property name="drive_wheel_height" value="-0.177505"/>
     <xacro:property name="support_wheel_height" value="-0.2252"/>
-    <xacro:macro name="Chassis" params="joints_movable:=true">
+    <xacro:macro name="Chassis" params="joints_movable:=true isaac:=false">
         <xacro:if value="${joints_movable}">
             <xacro:property name="wheel_joint_type" value="continuous"/>
@@ -154,4 +154,18 @@
             <origin xyz="0 0 0.11"/>
         </joint>
+        <link name="lidar_link">
+            <xacro:unless value="${isaac}">
+                <visual>
+                    <geometry>
+                        <mesh filename="file://$(find sensor_models)/meshes/orbbec/ms500.glb"/>
+                    </geometry>
+                </visual>
+            </xacro:unless>
+        </link>
+        <joint name="lidar_joint" type="fixed">
+            <origin xyz="0.24146 0  -0.14599"/>
+            <parent link="base_link"/>
+            <child link="lidar_link"/>
+        </joint>
     </xacro:macro>
 </robot>

File: xacro/chassis/linkhou_q1.xacro (robot description, xacro)
@@ -4,5 +4,5 @@
     <xacro:property name="drive_wheel_height" value="-0.220015"/>
     <xacro:property name="support_wheel_height" value="-0.253386"/>
-    <xacro:macro name="Chassis" params="joints_movable:=true">
+    <xacro:macro name="Chassis" params="joints_movable:=true isaac:=false">
         <xacro:if value="${joints_movable}">
             <xacro:property name="wheel_joint_type" value="continuous"/>
@@ -144,4 +144,46 @@
             <origin xyz="0 0 0.13"/>
         </joint>
+        <link name="chassis_front_camera">
+            <xacro:unless value="${isaac}">
+                <visual>
+                    <geometry>
+                        <mesh filename="file://$(find sensor_models)/meshes/orbbec/336.glb"/>
+                    </geometry>
+                </visual>
+            </xacro:unless>
+        </link>
+        <joint name="chassis_front_camera_joint" type="fixed">
+            <origin xyz="0.26 0.025 -0.02415" rpy="${PI/2} 0 ${PI/2}"/>
+            <parent link="base_link"/>
+            <child link="chassis_front_camera"/>
+        </joint>
+        <link name="chassis_back_camera">
+            <xacro:unless value="${isaac}">
+                <visual>
+                    <geometry>
+                        <mesh filename="file://$(find sensor_models)/meshes/orbbec/336.glb"/>
+                    </geometry>
+                </visual>
+            </xacro:unless>
+        </link>
+        <joint name="chassis_back_camera_joint" type="fixed">
+            <origin xyz="-0.30454 -0.025 -0.23529" rpy="${-PI*1/3} 0 ${PI/2}"/>
+            <parent link="base_link"/>
+            <child link="chassis_back_camera"/>
+        </joint>
+        <link name="lidar_link">
+            <xacro:unless value="${isaac}">
+                <visual>
+                    <geometry>
+                        <mesh filename="file://$(find sensor_models)/meshes/orbbec/ms500.glb"/>
+                    </geometry>
+                </visual>
+            </xacro:unless>
+        </link>
+        <joint name="lidar_joint" type="fixed">
+            <origin xyz="0.18694 0  -0.13232"/>
+            <parent link="base_link"/>
+            <child link="lidar_link"/>
+        </joint>
     </xacro:macro>
 </robot>

File: xacro/component.xacro (robot description, xacro)
@@ -9,5 +9,5 @@
     - arms: dual AR5 arms on arm_base (arms:=ar5_ccs / ar5_srs)
 -->
-<robot name="FiveAges_W1" xmlns:xacro="http://www.ros.org/wiki/xacro">
+<robot name="W1" xmlns:xacro="http://www.ros.org/wiki/xacro">
 	<xacro:property name="PI" value="3.1415926535897931"/>
 	<xacro:arg name="type" default="base"/>
@@ -16,11 +16,12 @@
 	<xacro:arg name="chassis_joints_movable" default="true"/>
 	<xacro:arg name="arms" default="ar5_srs"/>
+	<xacro:arg name="isaac" default="true"/>
 	<xacro:if value="${'$(arg type)' == 'base' and '$(arg chassis)' == 'w1'}">
 		<xacro:include filename="$(find fiveages_w1_description)/xacro/chassis/chassis.xacro"/>
-		<xacro:Chassis joints_movable="$(arg chassis_joints_movable)"/>
+		<xacro:Chassis joints_movable="$(arg chassis_joints_movable)" isaac="$(arg isaac)"/>
 	</xacro:if>
 	<xacro:if value="${'$(arg type)' == 'base' and '$(arg chassis)' == 'linkhou_q1'}">
 		<xacro:include filename="$(find fiveages_w1_description)/xacro/chassis/linkhou_q1.xacro"/>
-		<xacro:Chassis joints_movable="$(arg chassis_joints_movable)"/>
+		<xacro:Chassis joints_movable="$(arg chassis_joints_movable)"  isaac="$(arg isaac)"/>
 	</xacro:if>
 	<xacro:if value="${'$(arg type)' == 'linkhou_q1'}">

File: xacro/ros2_control/robot.xacro (robot description, xacro)
@@ -99,4 +99,5 @@
 		<gazebo>
 			<plugin filename="gz_ros2_control-system" name="gz_ros2_control::GazeboSimROS2ControlPlugin">
+				<parameters>$(find fiveages_w1_description)/config/ros2_control/common.yaml</parameters>
 				<parameters>$(find fiveages_w1_description)/config/ros2_control/ros2_controllers.yaml</parameters>
 				<xacro:if value="${left_gripper_type == 'rg75' or right_gripper_type == 'rg75'}">
