Commit message: ocs2 split body support

File: xacro/robot.xacro (robot description, xacro)
@@ -24,13 +24,19 @@
 	<!-- Body -->
 	<xacro:Body/>
+	<link name="arm_base"/>
+	<joint name="arm_base_joint" type="fixed">
+		<parent link="body_link4"/>
+		<child link="arm_base"/>
+		<origin xyz="0.0 0.0 0.41"/>
+	</joint>
 	<joint name="left_arm_mount" type="fixed">
-		<parent link="body_link4"/>
+		<parent link="arm_base"/>
 		<child link="left_base_link"/>
-		<origin xyz="0.0 0.12 0.41" rpy="-1.57 1.57 0"/>
+		<origin xyz="0.0 0.12 0" rpy="-1.57 1.57 0"/>
 	</joint>
 	<joint name="right_arm_mount" type="fixed">
-		<parent link="body_link4"/>
+		<parent link="arm_base"/>
 		<child link="right_base_link"/>
-		<origin xyz="0.0 -0.12 0.41" rpy="1.57 1.57 0"/>
+		<origin xyz="0.0 -0.12 0" rpy="1.57 1.57 0"/>
 	</joint>
 	<!-- Arms -->

Commit message: Type modify (#1)
* 修改了type相关 在type里同时写chassis和gripper

* 修复linkhou_rg75

* 将mpc_frequency从float转回integer

* 增加Linkhou & leapmotor的组合 urdf文件中的filename改成package形式

* 修改yaml文件gazebo的bug

* 修复ocs2中marker初始状态和eef不对齐

* ocs2 split body support

* add readme for split control

* ADD self collision config for rokae ar5 dual

---------

Co-authored-by: Zachary359 <zacharyx359@gmail.com>

File: xacro/robot.xacro (robot description, xacro)
@@ -2,7 +2,20 @@
 <robot name="FiveAges W1" xmlns:xacro="http://www.ros.org/wiki/xacro">
 	<!-- Arguments -->
-	<xacro:arg name="chassis" default="chassis"/>
+	<xacro:arg name="type" default=""/>
+	<xacro:arg name="collider" default="convex"/>
+	<!-- Select chassis & gripper based on type -->
+	<xacro:property name="type_arg" value="$(arg type)"/>
+	<xacro:property name="selected_chassis" value="chassis"/>
+	<xacro:property name="selected_gripper_type" value="${type_arg}"/>
+	<xacro:if value="${type_arg == 'linkhou_rg75'}">
+		<xacro:property name="selected_chassis" value="linkhou_q1"/>
+		<xacro:property name="selected_gripper_type" value="rg75"/>
+	</xacro:if>
+	<xacro:if value="${type_arg == 'linkhou_leapmotor'}">
+		<xacro:property name="selected_chassis" value="linkhou_q1"/>
+		<xacro:property name="selected_gripper_type" value="leapmotor"/>
+	</xacro:if>
 	<!-- Include Component Macros -->
-	<xacro:include filename="$(find fiveages_w1_description)/xacro/chassis/$(arg chassis).xacro"/>
+	<xacro:include filename="$(find fiveages_w1_description)/xacro/chassis/${selected_chassis}.xacro"/>
 	<xacro:include filename="$(find fiveages_w1_description)/xacro/body.xacro"/>
 	<xacro:include filename="$(find rokae_ar5_description)/xacro/arm.xacro"/>
@@ -11,18 +24,24 @@
 	<xacro:Chassis/>
 	<!-- Body -->
-	<xacro:Body/>
+	<xacro:Body collider="$(arg collider)"/>
+	<link name="arm_base"/>
+	<joint name="arm_base_joint" type="fixed">
+		<parent link="body_link4"/>
+		<child link="arm_base"/>
+		<origin xyz="0.0 0.0 0.41"/>
+	</joint>
 	<joint name="left_arm_mount" type="fixed">
-		<parent link="body_link4"/>
+		<parent link="arm_base"/>
 		<child link="left_base_link"/>
-		<origin xyz="0.0 0.12 0.41" rpy="-1.57 1.57 0"/>
+		<origin xyz="0.0 0.12 0" rpy="-1.57 1.57 0"/>
 	</joint>
 	<joint name="right_arm_mount" type="fixed">
-		<parent link="body_link4"/>
+		<parent link="arm_base"/>
 		<child link="right_base_link"/>
-		<origin xyz="0.0 -0.12 0.41" rpy="1.57 1.57 0"/>
+		<origin xyz="0.0 -0.12 0" rpy="1.57 1.57 0"/>
 	</joint>
 	<!-- Arms -->
-	<xacro:Arm name="left" direction="1"/>
-	<xacro:Arm name="right" direction="-1"/>
-	<xacro:Grippers/>
+	<xacro:Arm name="left" collider="$(arg collider)" direction="1"/>
+	<xacro:Arm name="right" collider="$(arg collider)" direction="-1"/>
+	<xacro:Grippers type="${selected_gripper_type}"/>
 </robot>

File: xacro/ros2_control/robot.xacro (robot description, xacro)
@@ -111,5 +111,5 @@
             <xacro:ar5_interfaces name="left"/>
             <xacro:ar5_interfaces name="right"/>
-            <xacro:if value="${'$(arg type)' == 'rg75' or '$(arg type)' == 'leapmotor'}">
+            <xacro:if value="${'$(arg type)' == 'rg75' or '$(arg type)' == 'leapmotor' or '$(arg type)' == 'linkhou_rg75' or '$(arg type)' == 'linkhou_leapmotor'}">
                 <xacro:include filename="$(find jodell_description)/xacro/ros2_control/RG75-300.xacro"/>
                 <xacro:rg75_interfaces name="left"/>
@@ -122,7 +122,20 @@
     <xacro:arg name="gazebo" default="false"/>
     <xacro:if value="$(arg gazebo)">
+        <xacro:property name="ros2_control_config_basename" value="ros2_controllers.yaml"/>
+        <xacro:if value="${type_arg == 'rg75'}">
+            <xacro:property name="ros2_control_config_basename" value="rg75.yaml"/>
+        </xacro:if>
+        <xacro:if value="${type_arg == 'leapmotor'}">
+            <xacro:property name="ros2_control_config_basename" value="leapmotor.yaml"/>
+        </xacro:if>
+        <xacro:if value="${type_arg == 'linkhou_rg75'}">
+            <xacro:property name="ros2_control_config_basename" value="linkhou_rg75.yaml"/>
+        </xacro:if>
+        <xacro:if value="${type_arg == 'linkhou_leapmotor'}">
+            <xacro:property name="ros2_control_config_basename" value="linkhou_leapmotor.yaml"/>
+        </xacro:if>
         <gazebo>
             <plugin filename="gz_ros2_control-system" name="gz_ros2_control::GazeboSimROS2ControlPlugin">
-                <parameters>$(find fiveages_w1_description)/config/ros2_control/ros2_controllers.yaml</parameters>
+                <parameters>$(find fiveages_w1_description)/config/ros2_control/${ros2_control_config_basename}</parameters>
             </plugin>
         </gazebo>

Commit message: fix robot xacro

File: xacro/robot.xacro (robot description, xacro)
@@ -65,10 +65,4 @@
 	<!-- Body -->
 	<xacro:Body collider="$(arg collider)"/>
-	<link name="arm_base"/>
-	<joint name="arm_base_joint" type="fixed">
-		<parent link="body_link4"/>
-		<child link="arm_base"/>
-		<origin xyz="0.0 0.0 0.41"/>
-	</joint>
 	<joint name="left_arm_mount" type="fixed">
 		<parent link="arm_base"/>
