Commit message: update w1 structure

File: xacro/chassis/chassis.xacro (robot description, xacro)
@@ -4,5 +4,11 @@
     <xacro:property name="drive_wheel_height" value="-0.177505"/>
     <xacro:property name="support_wheel_height" value="-0.2252"/>
-    <xacro:macro name="Chassis">
+    <xacro:macro name="Chassis" params="joints_movable:=true">
+        <xacro:if value="${joints_movable}">
+            <xacro:property name="wheel_joint_type" value="continuous"/>
+        </xacro:if>
+        <xacro:unless value="${joints_movable}">
+            <xacro:property name="wheel_joint_type" value="fixed"/>
+        </xacro:unless>
         <!-- Base Link -->
         <link name="base_footprint"/>
@@ -88,9 +94,11 @@
         </link>
         <!-- Left Wheel Joint -->
-        <joint name="chassis_left_joint" type="continuous">
+        <joint name="chassis_left_joint" type="${wheel_joint_type}">
             <origin xyz="-0.041 0.1846 ${drive_wheel_height}"/>
             <parent link="base_link"/>
             <child link="chassis_left_Link"/>
-            <axis xyz="0 1 0"/>
+            <xacro:if value="${joints_movable}">
+                <axis xyz="0 1 0"/>
+            </xacro:if>
         </joint>
         <!-- Right Wheel Link -->
@@ -120,9 +128,11 @@
         </link>
         <!-- Right Wheel Joint -->
-        <joint name="chassis_right_joint" type="continuous">
+        <joint name="chassis_right_joint" type="${wheel_joint_type}">
             <origin xyz="-0.041 -0.1846 ${drive_wheel_height}"/>
             <parent link="base_link"/>
             <child link="chassis_right_Link"/>
-            <axis xyz="0 1 0"/>
+            <xacro:if value="${joints_movable}">
+                <axis xyz="0 1 0"/>
+            </xacro:if>
         </joint>
         <link name="scan"/>

File: xacro/chassis/linkhou_q1.xacro (robot description, xacro)
@@ -4,5 +4,11 @@
     <xacro:property name="drive_wheel_height" value="-0.220015"/>
     <xacro:property name="support_wheel_height" value="-0.253386"/>
-    <xacro:macro name="Chassis">
+    <xacro:macro name="Chassis" params="joints_movable:=true">
+        <xacro:if value="${joints_movable}">
+            <xacro:property name="wheel_joint_type" value="continuous"/>
+        </xacro:if>
+        <xacro:unless value="${joints_movable}">
+            <xacro:property name="wheel_joint_type" value="fixed"/>
+        </xacro:unless>
         <!-- Base Link -->
         <link name="base_footprint"/>
@@ -86,9 +92,11 @@
             </collision>
         </link>
-        <joint name="chassis_left_joint" type="continuous">
+        <joint name="chassis_left_joint" type="${wheel_joint_type}">
             <origin xyz="-0.026651 0.20625 ${drive_wheel_height}"/>
             <parent link="base_link"/>
             <child link="left_wheel"/>
-            <axis xyz="0 1 0"/>
+            <xacro:if value="${joints_movable}">
+                <axis xyz="0 1 0"/>
+            </xacro:if>
         </joint>
         <link name="right_wheel">
@@ -116,9 +124,11 @@
             </collision>
         </link>
-        <joint name="chassis_right_joint" type="continuous">
+        <joint name="chassis_right_joint" type="${wheel_joint_type}">
             <origin xyz="-0.026651 -0.20625 ${drive_wheel_height}"/>
             <parent link="base_link"/>
             <child link="right_wheel"/>
-            <axis xyz="0 1 0"/>
+            <xacro:if value="${joints_movable}">
+                <axis xyz="0 1 0"/>
+            </xacro:if>
         </joint>
         <link name="scan"/>

File: xacro/component.xacro (robot description, xacro)
@@ -1,21 +1,58 @@
-<?xml version="1.0" ?>
-<!-- =================================================================================== -->
-<!-- |    Complete Robot Description for Agibot G1                                     | -->
-<!-- |    This file includes the base robot structure and both arms                    | -->
-<!-- =================================================================================== -->
+<?xml version="1.0"?>
+<!--
+  Component-wise description for FiveAges W1, used by
+  robot_common_launch/launch/visualize/component.launch.py
+  Supported types (arg "type"):
+    - base (default): chassis selected by chassis:=w1 / linkhou_q1
+    - linkhou_q1: alias for type:=base chassis:=linkhou_q1
+    - upper_body: trunk + head, rooted at base_link
+    - arms: dual AR5 arms on arm_base (arms:=ar5_ccs / ar5_srs)
+-->
 <robot name="FiveAges_W1" xmlns:xacro="http://www.ros.org/wiki/xacro">
+	<xacro:property name="PI" value="3.1415926535897931"/>
 	<xacro:arg name="type" default="base"/>
-	<xacro:if value="${'$(arg type)' == 'base'}">
+	<xacro:arg name="collider" default="convex"/>
+	<xacro:arg name="chassis" default="w1"/>
+	<xacro:arg name="chassis_joints_movable" default="true"/>
+	<xacro:arg name="arms" default="ar5_srs"/>
+	<xacro:if value="${'$(arg type)' == 'base' and '$(arg chassis)' == 'w1'}">
 		<xacro:include filename="$(find fiveages_w1_description)/xacro/chassis/chassis.xacro"/>
-		<xacro:Chassis />
+		<xacro:Chassis joints_movable="$(arg chassis_joints_movable)"/>
+	</xacro:if>
+	<xacro:if value="${'$(arg type)' == 'base' and '$(arg chassis)' == 'linkhou_q1'}">
+		<xacro:include filename="$(find fiveages_w1_description)/xacro/chassis/linkhou_q1.xacro"/>
+		<xacro:Chassis joints_movable="$(arg chassis_joints_movable)"/>
 	</xacro:if>
 	<xacro:if value="${'$(arg type)' == 'linkhou_q1'}">
 		<xacro:include filename="$(find fiveages_w1_description)/xacro/chassis/linkhou_q1.xacro"/>
-		<xacro:Chassis />
+		<xacro:Chassis joints_movable="$(arg chassis_joints_movable)"/>
 	</xacro:if>
 	<xacro:if value="${'$(arg type)' == 'upper_body'}">
 		<xacro:include filename="$(find fiveages_w1_description)/xacro/body.xacro"/>
 		<link name="base_link"/>
-		<xacro:Body/>
+		<xacro:Body collider="$(arg collider)"/>
+	</xacro:if>
+	<xacro:if value="${'$(arg type)' == 'arms'}">
+		<link name="arm_base"/>
+		<joint name="left_arm_mount" type="fixed">
+			<parent link="arm_base"/>
+			<child link="left_base_link"/>
+			<origin xyz="0.0 0.12 0" rpy="-${PI/2} ${PI/2} 0"/>
+		</joint>
+		<joint name="right_arm_mount" type="fixed">
+			<parent link="arm_base"/>
+			<child link="right_base_link"/>
+			<origin xyz="0.0 -0.12 0" rpy="${PI/2} ${PI/2} 0"/>
+		</joint>
+		<xacro:if value="${'$(arg arms)' == 'ar5_ccs'}">
+			<xacro:include filename="$(find ar5_ccs_description)/xacro/arm_ccs.xacro"/>
+			<xacro:AR5_CCS name="left" direction="1" collider="$(arg collider)"/>
+			<xacro:AR5_CCS name="right" direction="-1" collider="$(arg collider)"/>
+		</xacro:if>
+		<xacro:if value="${'$(arg arms)' == 'ar5_srs'}">
+			<xacro:include filename="$(find ar5_srs_description)/xacro/arm_srs.xacro"/>
+			<xacro:Arm name="left" direction="1" collider="$(arg collider)"/>
+			<xacro:Arm name="right" direction="-1" collider="$(arg collider)"/>
+		</xacro:if>
 	</xacro:if>
 </robot>

File: xacro/gazebo.xacro (robot description, xacro)
@@ -9,5 +9,5 @@
         <maxVel>10.0</maxVel>
     </gazebo>
-    <!-- Gazebo friction properties for left wheel -->
+    <!-- Native W1 chassis wheels -->
     <gazebo reference="chassis_left_Link">
         <mu1>1.0</mu1>
@@ -15,6 +15,16 @@
         <minDepth>0.0001</minDepth>
     </gazebo>
-    <!-- Gazebo friction properties for right wheel -->
     <gazebo reference="chassis_right_Link">
+        <mu1>1.0</mu1>
+        <mu2>1.0</mu2>
+        <minDepth>0.0001</minDepth>
+    </gazebo>
+    <!-- Linkhou Q1 chassis wheels -->
+    <gazebo reference="left_wheel">
+        <mu1>1.0</mu1>
+        <mu2>1.0</mu2>
+        <minDepth>0.0001</minDepth>
+    </gazebo>
+    <gazebo reference="right_wheel">
         <mu1>1.0</mu1>
         <mu2>1.0</mu2>

File: xacro/robot.xacro (robot description, xacro)
@@ -1,81 +1,92 @@
 <?xml version="1.0"?>
 <robot name="FiveAges W1" xmlns:xacro="http://www.ros.org/wiki/xacro">
-	<!-- Arguments -->
-	<xacro:arg name="type" default=""/>
-	<xacro:arg name="collider" default="convex"/>
-	<!-- Select chassis, arm & gripper based on type -->
-	<xacro:property name="type_arg" value="$(arg type)"/>
-	<xacro:property name="selected_chassis" value="chassis"/>
-	<xacro:property name="selected_arm" value="srs"/>
-	<xacro:property name="selected_gripper_type" value="${type_arg}"/>
-	<xacro:if value="${type_arg == 'linkhou_ccs_rg75'}">
-		<xacro:property name="selected_chassis" value="linkhou_q1"/>
-		<xacro:property name="selected_arm" value="ccs"/>
-		<xacro:property name="selected_gripper_type" value="rg75"/>
-	</xacro:if>
-	<xacro:if value="${type_arg == 'linkhou_srs_rg75'}">
-		<xacro:property name="selected_chassis" value="linkhou_q1"/>
-		<xacro:property name="selected_arm" value="srs"/>
-		<xacro:property name="selected_gripper_type" value="rg75"/>
-	</xacro:if>
-	<xacro:if value="${type_arg == 'linkhou_ccs_leapmotor'}">
-		<xacro:property name="selected_chassis" value="linkhou_q1"/>
-		<xacro:property name="selected_arm" value="ccs"/>
-		<xacro:property name="selected_gripper_type" value="leapmotor"/>
-	</xacro:if>
-	<xacro:if value="${type_arg == 'linkhou_srs_leapmotor'}">
-		<xacro:property name="selected_chassis" value="linkhou_q1"/>
-		<xacro:property name="selected_arm" value="srs"/>
-		<xacro:property name="selected_gripper_type" value="leapmotor"/>
-	</xacro:if>
-	<!-- Default chassis configurations -->
-	<xacro:if value="${type_arg == 'ccs_rg75'}">
-		<xacro:property name="selected_chassis" value="chassis"/>
-		<xacro:property name="selected_arm" value="ccs"/>
-		<xacro:property name="selected_gripper_type" value="rg75"/>
-	</xacro:if>
-	<xacro:if value="${type_arg == 'ccs_leapmotor'}">
-		<xacro:property name="selected_chassis" value="chassis"/>
-		<xacro:property name="selected_arm" value="ccs"/>
-		<xacro:property name="selected_gripper_type" value="leapmotor"/>
-	</xacro:if>
-	<xacro:if value="${type_arg == 'srs_rg75'}">
-		<xacro:property name="selected_chassis" value="chassis"/>
-		<xacro:property name="selected_arm" value="srs"/>
-		<xacro:property name="selected_gripper_type" value="rg75"/>
-	</xacro:if>
-	<xacro:if value="${type_arg == 'srs_leapmotor'}">
-		<xacro:property name="selected_chassis" value="chassis"/>
-		<xacro:property name="selected_arm" value="srs"/>
-		<xacro:property name="selected_gripper_type" value="leapmotor"/>
-	</xacro:if>
-	<!-- Include Component Macros -->
-	<xacro:include filename="$(find fiveages_w1_description)/xacro/chassis/${selected_chassis}.xacro"/>
-	<xacro:include filename="$(find fiveages_w1_description)/xacro/body.xacro"/>
-	<xacro:include filename="$(find fiveages_w1_description)/xacro/grippers.xacro"/>
-	<!-- Include Arm based on selected_arm -->
-	<xacro:if value="${selected_arm == 'ccs'}">
-		<xacro:include filename="$(find rokae_ar5_description)/xacro/arm_ccs.xacro"/>
-	</xacro:if>
-	<xacro:if value="${selected_arm == 'srs'}">
-		<xacro:include filename="$(find rokae_ar5_description)/xacro/arm_srs.xacro"/>
-	</xacro:if>
-	<!-- Chassis -->
-	<xacro:Chassis/>
-	<!-- Body -->
-	<xacro:Body collider="$(arg collider)"/>
-	<joint name="left_arm_mount" type="fixed">
-		<parent link="arm_base"/>
-		<child link="left_base_link"/>
-		<origin xyz="0.0 0.12 0" rpy="-1.57 1.57 0"/>
-	</joint>
-	<joint name="right_arm_mount" type="fixed">
-		<parent link="arm_base"/>
-		<child link="right_base_link"/>
-		<origin xyz="0.0 -0.12 0" rpy="1.57 1.57 0"/>
-	</joint>
-	<!-- Arms -->
-	<xacro:Arm name="left" collider="$(arg collider)" direction="1"/>
-	<xacro:Arm name="right" collider="$(arg collider)" direction="-1"/>
-	<xacro:Grippers type="${selected_gripper_type}"/>
+    <xacro:property name="PI" value="3.1415926535897931"/>
+    <xacro:arg name="collider" default="convex"/>
+    <!-- Native W1 chassis, or Linkhou Q1. Independent from the dual-arm kit. -->
+    <xacro:arg name="chassis" default="w1"/>
+    <!-- Same as W2: freeze wheels on the full robot. Component preview defaults to true. -->
+    <xacro:arg name="chassis_joints_movable" default="false"/>
+    <!-- Dual-arm kit: AR5 CCS v1 or AR5 SRS. CCS v2 is not used on W1. -->
+    <xacro:arg name="arms" default="ar5_srs"/>
+    <!-- End-effector selection:
+         - type is the symmetric default.
+         - left_type/right_type can override each side independently.
+         - eef_fixed_joints is used by OCS2 planning URDF generation. -->
+    <xacro:arg name="type" default=""/>
+    <xacro:arg name="left_type" default=""/>
+    <xacro:arg name="right_type" default=""/>
+    <xacro:arg name="eef_fixed_joints" default="false"/>
+    <xacro:arg name="left_tcp_offset_xyz" default="0 0 0"/>
+    <xacro:arg name="left_tcp_offset_rpy" default="0 0 0"/>
+    <xacro:arg name="right_tcp_offset_xyz" default="0 0 0"/>
+    <xacro:arg name="right_tcp_offset_rpy" default="0 0 0"/>
+    <xacro:property name="type_arg" value="$(arg type)"/>
+    <xacro:property name="left_type_arg" value="$(arg left_type)"/>
+    <xacro:property name="right_type_arg" value="$(arg right_type)"/>
+    <xacro:property name="effective_left_type" value="${left_type_arg if left_type_arg != '' else type_arg}"/>
+    <xacro:property name="effective_right_type" value="${right_type_arg if right_type_arg != '' else type_arg}"/>
+    <xacro:include filename="$(find ar5_ccs_description)/xacro/eef_type_resolver.xacro"/>
+    <xacro:set_side_eef_types side="left" type_key="${effective_left_type}"/>
+    <xacro:set_side_eef_types side="right" type_key="${effective_right_type}"/>
+    <xacro:property name="selected_hand_type" value="${left_hand_type if left_hand_type == right_hand_type else ''}"/>
+    <xacro:property name="selected_gripper_type" value="${left_gripper_type if left_gripper_type == right_gripper_type else ''}"/>
+    <xacro:property name="selected_gripper_pad" value="${left_gripper_pad if left_gripper_pad == right_gripper_pad else 'default'}"/>
+    <xacro:property name="chassis_arg" value="$(arg chassis)"/>
+    <xacro:if value="${chassis_arg == 'w1'}">
+        <xacro:include filename="$(find fiveages_w1_description)/xacro/chassis/chassis.xacro"/>
+        <xacro:Chassis joints_movable="$(arg chassis_joints_movable)"/>
+    </xacro:if>
+    <xacro:if value="${chassis_arg == 'linkhou_q1'}">
+        <xacro:include filename="$(find fiveages_w1_description)/xacro/chassis/linkhou_q1.xacro"/>
+        <xacro:Chassis joints_movable="$(arg chassis_joints_movable)"/>
+    </xacro:if>
+    <xacro:include filename="$(find fiveages_w1_description)/xacro/body.xacro"/>
+    <xacro:Body collider="$(arg collider)"/>
+    <joint name="left_arm_mount" type="fixed">
+        <parent link="arm_base"/>
+        <child link="left_base_link"/>
+        <origin xyz="0.0 0.12 0" rpy="-${PI/2} ${PI/2} 0"/>
+    </joint>
+    <joint name="right_arm_mount" type="fixed">
+        <parent link="arm_base"/>
+        <child link="right_base_link"/>
+        <origin xyz="0.0 -0.12 0" rpy="${PI/2} ${PI/2} 0"/>
+    </joint>
+    <xacro:if value="${'$(arg arms)' == 'ar5_ccs'}">
+        <xacro:include filename="$(find ar5_ccs_description)/xacro/arm_ccs.xacro"/>
+        <xacro:AR5_CCS name="left" direction="1" collider="$(arg collider)"/>
+        <xacro:AR5_CCS name="right" direction="-1" collider="$(arg collider)"/>
+    </xacro:if>
+    <xacro:if value="${'$(arg arms)' == 'ar5_srs'}">
+        <xacro:include filename="$(find ar5_srs_description)/xacro/arm_srs.xacro"/>
+        <xacro:Arm name="left" direction="1" collider="$(arg collider)"/>
+        <xacro:Arm name="right" direction="-1" collider="$(arg collider)"/>
+    </xacro:if>
+    <link name="left_tcp_offset"/>
+    <joint name="left_tcp_offset_joint" type="fixed">
+        <parent link="left_tcp"/>
+        <child link="left_tcp_offset"/>
+        <origin xyz="$(arg left_tcp_offset_xyz)" rpy="$(arg left_tcp_offset_rpy)"/>
+    </joint>
+    <link name="right_tcp_offset"/>
+    <joint name="right_tcp_offset_joint" type="fixed">
+        <parent link="right_tcp"/>
+        <child link="right_tcp_offset"/>
+        <origin xyz="$(arg right_tcp_offset_xyz)" rpy="$(arg right_tcp_offset_rpy)"/>
+    </joint>
+    <xacro:if value="${effective_left_type == 'robotiq85' or effective_right_type == 'robotiq85'}">
+        <xacro:include filename="$(find fiveages_w1_description)/xacro/grippers.xacro"/>
+        <xacro:Grippers type="robotiq85"/>
+    </xacro:if>
+    <xacro:unless value="${effective_left_type == 'robotiq85' or effective_right_type == 'robotiq85'}">
+        <xacro:include filename="$(find ar5_ccs_description)/xacro/eefs.xacro"/>
+        <xacro:EndEffectors
+            eef_fixed_joints="$(arg eef_fixed_joints)"
+            left_hand_type="${left_hand_type}"
+            left_gripper_type="${left_gripper_type}"
+            left_gripper_pad="${left_gripper_pad}"
+            right_hand_type="${right_hand_type}"
+            right_gripper_type="${right_gripper_type}"
+            right_gripper_pad="${right_gripper_pad}"/>
+    </xacro:unless>
 </robot>
