Commit message: 修改yaml文件gazebo的bug

File: xacro/ros2_control/robot.xacro (robot description, xacro)
@@ -7,17 +7,4 @@
     <xacro:include filename="$(find fiveages_w1_description)/xacro/ros2_control/body.xacro"/>
     <xacro:include filename="$(find fiveages_w1_description)/xacro/ros2_control/chassis.xacro"/>
-    <xacro:property name="ros2_control_config_basename" value="ros2_controllers.yaml"/>
-    <xacro:if value="${type_arg == 'rg75'}">
-        <xacro:property name="ros2_control_config_basename" value="rg75.yaml"/>
-    </xacro:if>
-    <xacro:if value="${type_arg == 'leapmotor'}">
-        <xacro:property name="ros2_control_config_basename" value="leapmotor.yaml"/>
-    </xacro:if>
-    <xacro:if value="${type_arg == 'linkhou_rg75'}">
-        <xacro:property name="ros2_control_config_basename" value="linkhou_rg75.yaml"/>
-    </xacro:if>
-    <xacro:if value="${type_arg == 'linkhou_leapmotor'}">
-        <xacro:property name="ros2_control_config_basename" value="linkhou_leapmotor.yaml"/>
-    </xacro:if>
     <xacro:if value="${'$(arg ros2_control_hardware_type)' == 'real'}">
         <ros2_control name="ar5_left_system" type="system">
@@ -88,4 +75,17 @@
     <xacro:arg name="gazebo" default="false"/>
     <xacro:if value="$(arg gazebo)">
+        <xacro:property name="ros2_control_config_basename" value="ros2_controllers.yaml"/>
+        <xacro:if value="${type_arg == 'rg75'}">
+            <xacro:property name="ros2_control_config_basename" value="rg75.yaml"/>
+        </xacro:if>
+        <xacro:if value="${type_arg == 'leapmotor'}">
+            <xacro:property name="ros2_control_config_basename" value="leapmotor.yaml"/>
+        </xacro:if>
+        <xacro:if value="${type_arg == 'linkhou_rg75'}">
+            <xacro:property name="ros2_control_config_basename" value="linkhou_rg75.yaml"/>
+        </xacro:if>
+        <xacro:if value="${type_arg == 'linkhou_leapmotor'}">
+            <xacro:property name="ros2_control_config_basename" value="linkhou_leapmotor.yaml"/>
+        </xacro:if>
         <gazebo>
             <plugin filename="gz_ros2_control-system" name="gz_ros2_control::GazeboSimROS2ControlPlugin">

Commit message: add config for dual arm with gripper

File: xacro/ros2_control/robot.xacro (robot description, xacro)
@@ -16,4 +16,12 @@
             </hardware>
             <xacro:ar5_interfaces name="left"/>
+            <xacro:if value="${'$(arg type)' == 'rg75'}">
+                <joint name="left_gripper_joint">
+                    <command_interface name="position"/>
+                    <state_interface name="position">
+                        <param name="initial_value">0</param>
+                    </state_interface>
+                </joint>
+            </xacro:if>
         </ros2_control>
         <ros2_control name="ar5_right_system" type="system">
@@ -25,4 +33,12 @@
             </hardware>
             <xacro:ar5_interfaces name="right"/>
+            <xacro:if value="${'$(arg type)' == 'rg75'}">
+                <joint name="right_gripper_joint">
+                    <command_interface name="position"/>
+                    <state_interface name="position">
+                        <param name="initial_value">0</param>
+                    </state_interface>
+                </joint>
+            </xacro:if>
         </ros2_control>
         <ros2_control name="eyou_body" type="system">
@@ -53,8 +69,16 @@
                 <plugin>rokae_ros2_control/RokaeHardware</plugin>
                 <param name="arm_ip">192.168.2.160</param>
-                <param name="joint_impedance">500,500,500,500,50,50,50</param>
+<!--                <param name="joint_impedance">500,500,500,500,50,50,50</param>-->
                 <param name="local_ip">192.168.2.233</param>
             </hardware>
             <xacro:ar5_interfaces name="left"/>
+            <xacro:if value="${'$(arg type)' == 'rg75'}">
+                <joint name="left_gripper_joint">
+                    <command_interface name="position"/>
+                    <state_interface name="position">
+                        <param name="initial_value">0</param>
+                    </state_interface>
+                </joint>
+            </xacro:if>
         </ros2_control>
         <ros2_control name="ar5_right_system" type="system">
@@ -66,4 +90,12 @@
             </hardware>
             <xacro:ar5_interfaces name="right"/>
+            <xacro:if value="${'$(arg type)' == 'rg75'}">
+                <joint name="right_gripper_joint">
+                    <command_interface name="position"/>
+                    <state_interface name="position">
+                        <param name="initial_value">0</param>
+                    </state_interface>
+                </joint>
+            </xacro:if>
         </ros2_control>
         <ros2_control name="eyou_body" type="system">

Commit message: add movej dialog

File: xacro/ros2_control/robot.xacro (robot description, xacro)
@@ -7,39 +7,41 @@
 	<xacro:include filename="$(find fiveages_w1_description)/xacro/ros2_control/body.xacro"/>
 	<xacro:include filename="$(find fiveages_w1_description)/xacro/ros2_control/chassis.xacro"/>
-    <xacro:if value="${'$(arg ros2_control_hardware_type)' == 'real'}">
-        <ros2_control name="ar5_left_system" type="system">
-            <hardware>
-                <plugin>rokae_ros2_control/RokaeHardware</plugin>
-                <param name="arm_ip">192.168.2.160</param>
-                <param name="joint_impedance">500,500,500,500,50,50,50</param>
-                <param name="local_ip">192.168.2.100</param>
-            </hardware>
-            <xacro:ar5_interfaces name="left"/>
-            <xacro:if value="${'$(arg type)' == 'rg75' or '$(arg type)' == 'ccs_rg75' or '$(arg type)' == 'srs_rg75' or '$(arg type)' == 'linkhou_rg75' or '$(arg type)' == 'linkhou_ccs_rg75' or '$(arg type)' == 'linkhou_srs_rg75'}">
-                <joint name="left_gripper_joint">
-                    <command_interface name="position"/>
-                    <state_interface name="position">
-                        <param name="initial_value">0</param>
-                    </state_interface>
-                </joint>
-            </xacro:if>
-        </ros2_control>
-        <ros2_control name="ar5_right_system" type="system">
-            <hardware>
-                <plugin>rokae_ros2_control/RokaeHardware</plugin>
-                <param name="arm_ip">192.168.2.161</param>
-                <param name="joint_impedance">500,500,500,500,50,50,50</param>
-                <param name="local_ip">192.168.2.100</param>
-            </hardware>
-            <xacro:ar5_interfaces name="right"/>
-            <xacro:if value="${'$(arg type)' == 'rg75' or '$(arg type)' == 'ccs_rg75' or '$(arg type)' == 'srs_rg75' or '$(arg type)' == 'linkhou_rg75' or '$(arg type)' == 'linkhou_ccs_rg75' or '$(arg type)' == 'linkhou_srs_rg75'}">
-                <joint name="right_gripper_joint">
-                    <command_interface name="position"/>
-                    <state_interface name="position">
-                        <param name="initial_value">0</param>
-                    </state_interface>
-                </joint>
-            </xacro:if>
-        </ros2_control>
+	<xacro:if value="${'$(arg ros2_control_hardware_type)' == 'real'}">
+		<ros2_control name="ar5_left_system" type="system">
+			<hardware>
+				<plugin>rokae_ros2_control/RokaeHardware</plugin>
+				<param name="arm_ip">192.168.2.160</param>
+				<param name="joint_impedance">500,500,500,500,50,50,50</param>
+				<param name="local_ip">192.168.2.100</param>
+			</hardware>
+			<xacro:ar5_interfaces name="left"/>
+			<xacro:if
+					value="${'$(arg type)' == 'rg75' or '$(arg type)' == 'ccs_rg75' or '$(arg type)' == 'srs_rg75' or '$(arg type)' == 'linkhou_rg75' or '$(arg type)' == 'linkhou_ccs_rg75' or '$(arg type)' == 'linkhou_srs_rg75'}">
+				<joint name="left_gripper_joint">
+					<command_interface name="position"/>
+					<state_interface name="position">
+						<param name="initial_value">0</param>
+					</state_interface>
+				</joint>
+			</xacro:if>
+		</ros2_control>
+		<ros2_control name="ar5_right_system" type="system">
+			<hardware>
+				<plugin>rokae_ros2_control/RokaeHardware</plugin>
+				<param name="arm_ip">192.168.2.161</param>
+				<param name="joint_impedance">500,500,500,500,50,50,50</param>
+				<param name="local_ip">192.168.2.100</param>
+			</hardware>
+			<xacro:ar5_interfaces name="right"/>
+			<xacro:if
+					value="${'$(arg type)' == 'rg75' or '$(arg type)' == 'ccs_rg75' or '$(arg type)' == 'srs_rg75' or '$(arg type)' == 'linkhou_rg75' or '$(arg type)' == 'linkhou_ccs_rg75' or '$(arg type)' == 'linkhou_srs_rg75'}">
+				<joint name="right_gripper_joint">
+					<command_interface name="position"/>
+					<state_interface name="position">
+						<param name="initial_value">0</param>
+					</state_interface>
+				</joint>
+			</xacro:if>
+		</ros2_control>
 		<ros2_control name="eyou_body" type="system">
 			<hardware>
@@ -64,39 +66,41 @@
 		</ros2_control>
 	</xacro:if>
-    <xacro:if value="${'$(arg ros2_control_hardware_type)' == 'real-laptop'}">
-        <ros2_control name="ar5_left_system" type="system">
-            <hardware>
-                <plugin>rokae_ros2_control/RokaeHardware</plugin>
-                <param name="arm_ip">192.168.2.160</param>
-<!--                <param name="joint_impedance">500,500,500,500,50,50,50</param>-->
-                <param name="local_ip">192.168.2.233</param>
-            </hardware>
-            <xacro:ar5_interfaces name="left"/>
-            <xacro:if value="${'$(arg type)' == 'rg75' or '$(arg type)' == 'ccs_rg75' or '$(arg type)' == 'srs_rg75' or '$(arg type)' == 'linkhou_rg75' or '$(arg type)' == 'linkhou_ccs_rg75' or '$(arg type)' == 'linkhou_srs_rg75'}">
-                <joint name="left_gripper_joint">
-                    <command_interface name="position"/>
-                    <state_interface name="position">
-                        <param name="initial_value">0</param>
-                    </state_interface>
-                </joint>
-            </xacro:if>
-        </ros2_control>
-        <ros2_control name="ar5_right_system" type="system">
-            <hardware>
-                <plugin>rokae_ros2_control/RokaeHardware</plugin>
-                <param name="arm_ip">192.168.2.161</param>
-                <param name="joint_impedance">500,500,500,500,50,50,50</param>
-                <param name="local_ip">192.168.2.233</param>
-            </hardware>
-            <xacro:ar5_interfaces name="right"/>
-            <xacro:if value="${'$(arg type)' == 'rg75' or '$(arg type)' == 'ccs_rg75' or '$(arg type)' == 'srs_rg75' or '$(arg type)' == 'linkhou_rg75' or '$(arg type)' == 'linkhou_ccs_rg75' or '$(arg type)' == 'linkhou_srs_rg75'}">
-                <joint name="right_gripper_joint">
-                    <command_interface name="position"/>
-                    <state_interface name="position">
-                        <param name="initial_value">0</param>
-                    </state_interface>
-                </joint>
-            </xacro:if>
-        </ros2_control>
+	<xacro:if value="${'$(arg ros2_control_hardware_type)' == 'real-laptop'}">
+		<ros2_control name="ar5_left_system" type="system">
+			<hardware>
+				<plugin>rokae_ros2_control/RokaeHardware</plugin>
+				<param name="arm_ip">192.168.2.160</param>
+				<!--                <param name="joint_impedance">500,500,500,500,50,50,50</param>-->
+				<param name="local_ip">192.168.2.233</param>
+			</hardware>
+			<xacro:ar5_interfaces name="left"/>
+			<xacro:if
+					value="${'$(arg type)' == 'rg75' or '$(arg type)' == 'ccs_rg75' or '$(arg type)' == 'srs_rg75' or '$(arg type)' == 'linkhou_rg75' or '$(arg type)' == 'linkhou_ccs_rg75' or '$(arg type)' == 'linkhou_srs_rg75'}">
+				<joint name="left_gripper_joint">
+					<command_interface name="position"/>
+					<state_interface name="position">
+						<param name="initial_value">0</param>
+					</state_interface>
+				</joint>
+			</xacro:if>
+		</ros2_control>
+		<ros2_control name="ar5_right_system" type="system">
+			<hardware>
+				<plugin>rokae_ros2_control/RokaeHardware</plugin>
+				<param name="arm_ip">192.168.2.161</param>
+				<param name="joint_impedance">500,500,500,500,50,50,50</param>
+				<param name="local_ip">192.168.2.233</param>
+			</hardware>
+			<xacro:ar5_interfaces name="right"/>
+			<xacro:if
+					value="${'$(arg type)' == 'rg75' or '$(arg type)' == 'ccs_rg75' or '$(arg type)' == 'srs_rg75' or '$(arg type)' == 'linkhou_rg75' or '$(arg type)' == 'linkhou_ccs_rg75' or '$(arg type)' == 'linkhou_srs_rg75'}">
+				<joint name="right_gripper_joint">
+					<command_interface name="position"/>
+					<state_interface name="position">
+						<param name="initial_value">0</param>
+					</state_interface>
+				</joint>
+			</xacro:if>
+		</ros2_control>
 		<ros2_control name="eyou_body" type="system">
 			<hardware>
@@ -145,54 +149,55 @@
 				<xacro:ar5_interfaces name="left"/>
 				<xacro:ar5_interfaces name="right"/>
-            <xacro:if value="${'$(arg type)' == 'rg75' or '$(arg type)' == 'leapmotor' or '$(arg type)' == 'linkhou_rg75' or '$(arg type)' == 'linkhou_leapmotor' or '$(arg type)' == 'ccs_rg75' or '$(arg type)' == 'ccs_leapmotor' or '$(arg type)' == 'srs_rg75' or '$(arg type)' == 'srs_leapmotor' or '$(arg type)' == 'linkhou_ccs_rg75' or '$(arg type)' == 'linkhou_ccs_leapmotor' or '$(arg type)' == 'linkhou_srs_rg75' or '$(arg type)' == 'linkhou_srs_leapmotor'}">
-                <xacro:include filename="$(find jodell_description)/xacro/ros2_control/RG75-300.xacro"/>
-                <xacro:rg75_interfaces name="left"/>
-                <xacro:rg75_interfaces name="right"/>
-            </xacro:if>
-        </ros2_control>
-        </xacro:unless>
-    </xacro:unless>
+				<xacro:if
+						value="${'$(arg type)' == 'rg75' or '$(arg type)' == 'leapmotor' or '$(arg type)' == 'linkhou_rg75' or '$(arg type)' == 'linkhou_leapmotor' or '$(arg type)' == 'ccs_rg75' or '$(arg type)' == 'ccs_leapmotor' or '$(arg type)' == 'srs_rg75' or '$(arg type)' == 'srs_leapmotor' or '$(arg type)' == 'linkhou_ccs_rg75' or '$(arg type)' == 'linkhou_ccs_leapmotor' or '$(arg type)' == 'linkhou_srs_rg75' or '$(arg type)' == 'linkhou_srs_leapmotor'}">
+					<xacro:include filename="$(find jodell_description)/xacro/ros2_control/RG75-300.xacro"/>
+					<xacro:rg75_interfaces name="left"/>
+					<xacro:rg75_interfaces name="right"/>
+				</xacro:if>
+			</ros2_control>
+		</xacro:unless>
+	</xacro:unless>
 	<!-- Gazebo plugin configuration -->
 	<xacro:arg name="gazebo" default="false"/>
 	<xacro:if value="$(arg gazebo)">
 		<xacro:property name="ros2_control_config_basename" value="ros2_controllers.yaml"/>
-        <!-- Default chassis configurations -->
-        <xacro:if value="${type_arg == 'rg75'}">
-            <xacro:property name="ros2_control_config_basename" value="rg75.yaml"/>
-        </xacro:if>
+		<!-- Default chassis configurations -->
+		<xacro:if value="${type_arg == 'rg75'}">
+			<xacro:property name="ros2_control_config_basename" value="rg75.yaml"/>
+		</xacro:if>
 		<xacro:if value="${type_arg == 'leapmotor'}">
 			<xacro:property name="ros2_control_config_basename" value="leapmotor.yaml"/>
 		</xacro:if>
-        <xacro:if value="${type_arg == 'ccs_rg75'}">
-            <xacro:property name="ros2_control_config_basename" value="ccs_rg75.yaml"/>
-        </xacro:if>
-        <xacro:if value="${type_arg == 'ccs_leapmotor'}">
-            <xacro:property name="ros2_control_config_basename" value="ccs_leapmotor.yaml"/>
-        </xacro:if>
-        <xacro:if value="${type_arg == 'srs_rg75'}">
-            <xacro:property name="ros2_control_config_basename" value="srs_rg75.yaml"/>
-        </xacro:if>
-        <xacro:if value="${type_arg == 'srs_leapmotor'}">
-            <xacro:property name="ros2_control_config_basename" value="srs_leapmotor.yaml"/>
-        </xacro:if>
-        <!-- Linkhou chassis configurations -->
-        <xacro:if value="${type_arg == 'linkhou_rg75'}">
-            <xacro:property name="ros2_control_config_basename" value="linkhou_rg75.yaml"/>
-        </xacro:if>
-        <xacro:if value="${type_arg == 'linkhou_leapmotor'}">
-            <xacro:property name="ros2_control_config_basename" value="linkhou_leapmotor.yaml"/>
-        </xacro:if>
-        <xacro:if value="${type_arg == 'linkhou_ccs_rg75'}">
-            <xacro:property name="ros2_control_config_basename" value="linkhou_ccs_rg75.yaml"/>
-        </xacro:if>
-        <xacro:if value="${type_arg == 'linkhou_ccs_leapmotor'}">
-            <xacro:property name="ros2_control_config_basename" value="linkhou_ccs_leapmotor.yaml"/>
-        </xacro:if>
-        <xacro:if value="${type_arg == 'linkhou_srs_rg75'}">
-            <xacro:property name="ros2_control_config_basename" value="linkhou_srs_rg75.yaml"/>
-        </xacro:if>
-        <xacro:if value="${type_arg == 'linkhou_srs_leapmotor'}">
-            <xacro:property name="ros2_control_config_basename" value="linkhou_srs_leapmotor.yaml"/>
-        </xacro:if>
+		<xacro:if value="${type_arg == 'ccs_rg75'}">
+			<xacro:property name="ros2_control_config_basename" value="ccs_rg75.yaml"/>
+		</xacro:if>
+		<xacro:if value="${type_arg == 'ccs_leapmotor'}">
+			<xacro:property name="ros2_control_config_basename" value="ccs_leapmotor.yaml"/>
+		</xacro:if>
+		<xacro:if value="${type_arg == 'srs_rg75'}">
+			<xacro:property name="ros2_control_config_basename" value="srs_rg75.yaml"/>
+		</xacro:if>
+		<xacro:if value="${type_arg == 'srs_leapmotor'}">
+			<xacro:property name="ros2_control_config_basename" value="srs_leapmotor.yaml"/>
+		</xacro:if>
+		<!-- Linkhou chassis configurations -->
+		<xacro:if value="${type_arg == 'linkhou_rg75'}">
+			<xacro:property name="ros2_control_config_basename" value="linkhou_rg75.yaml"/>
+		</xacro:if>
+		<xacro:if value="${type_arg == 'linkhou_leapmotor'}">
+			<xacro:property name="ros2_control_config_basename" value="linkhou_leapmotor.yaml"/>
+		</xacro:if>
+		<xacro:if value="${type_arg == 'linkhou_ccs_rg75'}">
+			<xacro:property name="ros2_control_config_basename" value="linkhou_ccs_rg75.yaml"/>
+		</xacro:if>
+		<xacro:if value="${type_arg == 'linkhou_ccs_leapmotor'}">
+			<xacro:property name="ros2_control_config_basename" value="linkhou_ccs_leapmotor.yaml"/>
+		</xacro:if>
+		<xacro:if value="${type_arg == 'linkhou_srs_rg75'}">
+			<xacro:property name="ros2_control_config_basename" value="linkhou_srs_rg75.yaml"/>
+		</xacro:if>
+		<xacro:if value="${type_arg == 'linkhou_srs_leapmotor'}">
+			<xacro:property name="ros2_control_config_basename" value="linkhou_srs_leapmotor.yaml"/>
+		</xacro:if>
 		<gazebo>
 			<plugin filename="gz_ros2_control-system" name="gz_ros2_control::GazeboSimROS2ControlPlugin">
